File: builds/6s/50A/CAN_485_faraday/kicad/open_secure_esc_6s_50a_can485_faraday.kicad_sch (KiCad schematic)
At the start: 0 parts

Commit message: Populate 6S/50A CAN+RS485/Faraday KiCad project (schematic, .kicad_pro, PCB)
Generates the previously-empty schematic skeleton into a fully wired,
44-symbol schematic on a centered A0 sheet: every documented MCU pin
assignment (symbols/specs/MSPM0G3507.json) is routed with real wires to
its peer chip, shared rails (GND/VM/3V3/VREF_MID/isolated grounds/phase
nodes) use same-name global labels with a wire stub at each pin. Title
block company is Griffing Technology LLC. Generic support passives
(decoupling, pull-ups, bias dividers) use KiCad's standard Device/
Connector_Generic parts, flagged as engineering defaults rather than
datasheet-sourced. Genuinely open design questions from README.md
(DRV8353S-vs-INA240 current sense, nFAULT routing, isolated supply
sourcing, 3V3 regulator selection) are left open on the sheet rather
than silently resolved.

Adds a hand-authored .kicad_pro and a .kicad_pcb with footprints placed
for every BOM part with a confirmed footprint, plus a centered board
outline on A3; DRV8353S (no confirmed footprint) gets a reserved-area
marker instead of a fabricated footprint. No netlist import or routing
yet -- see kicad/README.md for exact status and next steps.

Adds builds/6s/50A/CAN_485_faraday/kicad/tools/ (gen_schematic.py,
gen_pcb.py, genlib.py) as the reproducible generators for both files,
mirroring symbols/tools/gen_kicad_symbol.py. Also fixes sym-lib-table
(was missing the WE_SHC_3670375 frame) and adds Device/Connector_Generic
entries for the generic parts.

Co-Authored-By: Claude Sonnet 5 <noreply@anthropic.com>
Claude-Session: https://claude.ai/code/session_011fHSpdvtPAVWjNqNm1QQuM
Parts:
- added BT1, BT2, BT3, BT4, BT5, BT6: INR-21700-P42A, symbol INR21700_P42A:INR21700_P42A
- added C1: 100uF/50V, Capacitor_THT:CP_Radial_D10.0mm_P5.00mm, symbol Device:C_Polarized
- added C2, C3, C6: 100nF, Capacitor_SMD:C_0805_2012Metric, symbol Device:C
- added C4: 2.2nF, Capacitor_SMD:C_0805_2012Metric, symbol Device:C
- added C5, C7, C8: 1uF, Capacitor_SMD:C_0805_2012Metric, symbol Device:C
- added J1: J_SWD, Connector_PinHeader_2.54mm:PinHeader_1x04_P2.54mm_Vertical, symbol Connector_Generic:Conn_01x04
- added J2: J_CAN, Connector_PinHeader_2.54mm:PinHeader_1x02_P2.54mm_Vertical, symbol Connector_Generic:Conn_01x02
- added J3: J_RS485, Connector_PinHeader_2.54mm:PinHeader_1x02_P2.54mm_Vertical, symbol Connector_Generic:Conn_01x02
- added J4: J_MOTOR, Connector_PinHeader_2.54mm:PinHeader_1x03_P2.54mm_Vertical, symbol Connector_Generic:Conn_01x03
- added Q1, Q2, Q3, Q4, Q5, Q6: IRFB4110PBF, Package_TO_SOT_THT:TO-220-3_Vertical, symbol IRFB4110PBF:IRFB4110PBF
- added R1, R10, R2, R3, R7, R8: 10k, Resistor_SMD:R_0805_2012Metric, symbol Device:R
- added R4, R5, R6: 1mOhm, Resistor_SMD:R_2512_6332Metric, symbol WSLP2512:WSLP2512
- added R9: 90k, Resistor_SMD:R_0805_2012Metric, symbol Device:R
- added SH1: WE-SHC 3671375 (cover), symbol WE_SHC_3671375:WE_SHC_3671375
- added SH2: WE-SHC 3670375 (frame), symbol WE_SHC_3670375:WE_SHC_3670375
- added U1: MSPM0G3507SPMR, Package_QFP:LQFP-64_10x10mm_P0.5mm, symbol MSPM0G3507:MSPM0G3507
- added U2: SLB9672, Package_DFN_QFN:QFN-32-1EP_5x5mm_P0.5mm, symbol SLB9672:SLB9672
- added U3: ADM3055E/ADM3057E, Package_SO:SOIC-20W_7.5x12.8mm_P1.27mm, symbol ADM3055E_ADM3057E:ADM3055E_ADM3057E
- added U4: ADM2582E/ADM2587E, Package_SO:SOIC-20W_7.5x12.8mm_P1.27mm, symbol ADM2582E_ADM2587E:ADM2582E_ADM2587E
- added U5: DRV8353S, symbol DRV8353S:DRV8353S
- added U6, U7, U8: INA240, Package_SO:SOIC-8_3.9x4.9mm_P1.27mm, symbol INA240:INA240
Connections:
- new net: BT1.2 (-), BT2.1 (+)
- new net: Q5.1 (G), Q6.1 (G), U5.16 (GHC), U5.18 (GLC)
- new net: R3.2, U5.26 (nFAULT)
- new net: U1.10 (GD_SPI_SCK), U1.11 (GD_SPI_MOSI), U1.30 (GD_SPI_CS), U1.33 (PWM_AH), U1.34 (PWM_AL), U1.35 (PWM_CH), U1.47 (PWM_BH), U1.48 (PWM_BL), U1.51 (PWM_CL), U5.28 (SDI), U5.29 (SCLK), U5.30 (nSCS), U5.32 (INHA), U5.33 (INLA), U5.34 (INHB), U5.35 (INLB), U5.36 (INHC), U5.37 (INLC)
- new net: BT2.2 (-), BT3.1 (+)
- new net: BT3.2 (-), BT4.1 (+)
- new net: U1.64 (RS485_TXD), U4.7 (TxD)
- new net: BT4.2 (-), BT5.1 (+)
- new net: BT5.2 (-), BT6.1 (+)
- new net: U1.42 (TPM_SPI_CS), U1.45 (TPM_SPI_MOSI), U1.46 (TPM_SPI_SCK), U1.59 (TPM_RST#), U2.17 (RST#), U2.19 (SCLK), U2.20 (CS#), U2.21 (MOSI)
- new net: U1.44 (TPM_SPI_MISO), U1.58 (TPM_PIRQ#), U2.18 (PIRQ#), U2.24 (MISO)
- new net: U1.5 (CAN_TX), U3.7 (TXD)
- new net 3V3: C3.1, J1.3 (Pin_3), R1.1, R2.1, R2.2, R3.1, R7.1, U1.40 (VDD), U1.9 (GD_SPI_MISO), U2.1 (VDD), U2.10 (NCI/VDD), U2.14 (VDD), U2.22 (VDD), U2.8 (NCI/VDD), U3.3 (VCC), U3.4 (VIO), U4.2 (VCC), U4.8 (VCC), U5.27 (SDO), U5.31 (ENABLE), U6.6 (VS), U7.6 (VS), U8.6 (VS)
- new net ADC_IU: U1.31 (ADC_IU), U6.5 (OUT)
- new net ADC_IV: U1.26 (ADC_IV), U7.5 (OUT)
- new net ADC_IW: U1.25 (ADC_IW), U8.5 (OUT)
- new net CAN_ISO_GND: BT6.2 (-), C1.2 (-), C2.1, C2.2, C3.2, C6.1, C6.2, C7.1, C7.2, C8.1, C8.2, J1.1 (Pin_1), J1.2 (Pin_2), J1.4 (Pin_4), J2.1 (Pin_1), J2.2 (Pin_2), R1.2, R10.2, R4.2, R5.2, R6.2, R8.2, SH1.1 (SHIELD_GND), SH2.1 (SHIELD_GND), U1.12 (SWDIO), U1.13 (SWCLK), U1.32 (VCORE), U1.38 (NRST), U1.41 (VSS), U1.6 (CAN_RX), U2.16 (NCI/GND), U2.2 (GND), U2.23 (GND), U2.32 (GND), U2.9 (GND), U3.1 (GND1), U3.10 (GND1), U3.11 (GND2), U3.12 (RS), U3.13 (CANL), U3.14 (CANH), U3.15 (GND2), U3.16 (VISOIN), U3.18 (GNDISO), U3.2 (GND1), U3.20 (GNDISO), U3.5 (RXD), U3.6 (SILENT), U3.8 (STBY), U4.1 (GND1), U4.10 (GND1), U4.3 (GND1), U4.9 (GND1), U5.10 (SNA), U5.11 (SNB), U5.20 (SNC), U5.24 (VREF), U5.25 (AGND), U5.38 (DVDD), U5.39 (GND), U5.40 (VGLS), U6.1 (IN-), U6.2 (GND), U7.1 (IN-), U7.2 (GND), U8.1 (IN-), U8.2 (GND)
- new net CAN_VISOOUT: U3.19 (VISOOUT)
- new net ISENSE_A_HI: Q1.1 (G), Q2.1 (G), Q2.3 (S), Q3.1 (G), Q4.1 (G), Q4.3 (S), R4.1, R5.1, U5.12 (SPB), U5.13 (GLB), U5.15 (GHB), U5.6 (GHA), U5.8 (GLA), U5.9 (SPA), U6.8 (IN+), U7.8 (IN+)
- new net ISENSE_C_HI: Q6.3 (S), R6.1, U5.19 (SPC), U8.8 (IN+)
- new net PH_A: J4.1 (Pin_1), Q1.3 (S), Q2.2 (D), U5.7 (SHA)
- new net PH_B: J4.2 (Pin_2), Q3.3 (S), Q4.2 (D), U5.14 (SHB)
- new net PH_C: J4.3 (Pin_3), Q5.3 (S), Q6.2 (D), U5.17 (SHC)
- new net RS485_A: J3.1 (Pin_1), J3.2 (Pin_2), U4.13 (Y), U4.15 (Z), U4.17 (B), U4.18 (A)
- new net RS485_DE_RE: U1.36 (RS485_DE_RE), U4.5 (RE), U4.6 (DE)
- new net RS485_ISO_GND: U1.1 (RS485_RXD), U4.11 (GND2), U4.14 (GND2), U4.16 (GND2), U4.20 (GND2), U4.4 (RxD)
- new net RS485_VISOIN_OPEN: U4.19 (VISOIN)
- new net RS485_VISOOUT: U4.12 (VISOOUT)
- new net VBUS_SENSE: R10.1, R9.2, U1.8 (ADC_VBUS)
- new net VM: BT1.1 (+), C1.1 (+), C4.1, C4.2, C5.1, C5.2, Q1.2 (D), Q3.2 (D), Q5.2 (D), R9.1, U5.1 (CPL), U5.2 (CPH), U5.3 (VM), U5.4 (VDRAIN), U5.5 (VCP)
- new net VREF_MID: R7.2, R8.1, U6.3 (REF2), U6.7 (REF1), U7.3 (REF2), U7.7 (REF1), U8.3 (REF2), U8.7 (REF1)
- no-connect marks 0 -> 24
Other:
- note added: "Battery pack -- 6S (Molicel INR-21700-P42A x6 series), REFERENCES.md [14]"
- note added: "Faraday shield (WE-SHC 3671375 cover + 3670375 frame) over gate-drive / high-di/dt switching-node area -- see ../README.md EMI Hardening tier"
- note added: "SOA/SOB/SOC (DRV8353S integrated per-phase CSA outputs) intentionally left unconnected: this build routes ADC_IU/IV/IW from external INA240 devices instead -- DRV8353S-vs-INA240 current-sense sourcing is an open design question, see ../README.md Open items."
- note added: "nFAULT: pulled up only, not wired to MCU in this build -- open item, see ../README.md"
- company: Open-Secure-ESC project (CERN-OHL-P v2) -> Griffing Technology LLC

Commit message: Fix ERC power-pin-not-driven violations and ruff/CI version mismatch
CI's ERC check (real KiCad 9.0 via kicad-cli sch erc) flagged 8 error-
severity violations: every rail that's carried only by same-name global
labels with no regulator/source symbol on the sheet (GND, 3V3, VM, the
two isolated-transceiver grounds, the two open isolated-supply nets)
plus DRV8353S.VREF (wired only to its own decoupling cap, no label at
all) has power-input pins with no declared driver. Added a PWR_FLAG
generic part (genlib.py power:PWR_FLAG) and placed one on each of those
8 nets -- KiCad's standard mechanism for "this net is intentionally
driven from outside this schematic," not a claim about where the power
actually comes from (the 3V3 regulator and isolated-supply sourcing
are still open items, documented as such). Traced every power_in-typed
pin across every part spec to confirm these 8 are the complete set.
Verified with kicad-cli sch export svg/netlist (can't run sch erc
directly -- KiCad 7.0.11, the newest available via apt here, predates
that subcommand) and a wire-connectivity/net-conflict re-check.

Also fixes a ruff version mismatch that broke the previous lint fix:
this sandbox has two ruff installs (0.15.8 pre-existing, 0.16.1 from
this session's pip install) that disagree on whether E402 is
default-enabled, and CI's fresh `pip install ruff` matches 0.16.1's
behavior (confirmed from the actual CI log: "non-enabled: E402"). The
`# noqa: E402` comments added in the previous commit were therefore
themselves flagged as unused directives (RUF100) under CI's real ruff.
Removed them and re-ran ruff check --fix / ruff format under the
0.16.1 binary specifically to match CI.

Co-Authored-By: Claude Sonnet 5 <noreply@anthropic.com>
Claude-Session: https://claude.ai/code/session_011fHSpdvtPAVWjNqNm1QQuM
Parts:
- added FLG1, FLG2, FLG3, FLG4, FLG5, FLG6, FLG7, FLG8: PWR_FLAG, symbol power:PWR_FLAG
Connections:
- net 3V3: now also FLG2.1 (pwr)
- net CAN_ISO_GND: now also FLG1.1 (pwr), FLG4.1 (pwr), FLG6.1 (pwr), FLG8.1 (pwr)
- net RS485_ISO_GND: now also FLG5.1 (pwr)
- net RS485_VISOIN_OPEN: now also FLG7.1 (pwr)
- net VM: now also FLG3.1 (pwr)
Changed lines of the file:
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@@
+    (stroke (width 0) (type default))
+  )
+  (wire (pts (xy 99.85 324.07) (xy 99.85 325.72))
+    (stroke (width 0) (type default))
+  )
+  (wire (pts (xy 469.85 191.37) (xy 469.85 193.02))
+    (stroke (width 0) (type default))
+  )
+  (wire (pts (xy 99.85 61.37) (xy 99.85 63.02))
+    (stroke (width 0) (type default))
+  )
+  (wire (pts (xy 380.01 236.29) (xy 380.01 237.94))
+    (stroke (width 0) (type default))
+  )
+  (wire (pts (xy 380.01 453.75) (xy 380.01 455.4))
+    (stroke (width 0) (type default))
+  )
+  (wire (pts (xy 380.01 246.45) (xy 380.01 248.1))
+    (stroke (width 0) (type default))
+  )
+  (wire (pts (xy 380.01 474.07) (xy 380.01 475.72))
+    (stroke (width 0) (type default))
+  )
+  (wire (pts (xy 721.12 487.4) (xy 721.12 489.05))
     (stroke (width 0) (type default))
   )
@@
       (effects (font (size 1.27 1.27)) hide)
     )
+    (pin "1")
+  )
+  (symbol (lib_id "power:PWR_FLAG") (at 99.85 317.72 0) (unit 1)
+    (in_bom yes) (on_board yes)
+    (property "Reference" "FLG1" (id 0) (at 99.85 308.83 0)
+      (effects (font (size 1.27 1.27)))
+    )
+    (property "Value" "PWR_FLAG" (id 1) (at 99.85 311.37 0)
+      (effects (font (size 1.27 1.27)))
+    )
+    (property "Footprint" "" (id 2) (at 99.85 317.72 0)
+      (effects (font (size 1.27 1.27)) hide)
+    )
+    (property "Datasheet" "" (id 3) (at 99.85 317.72 0)
+      (effects (font (size 1.27 1.27)) hide)
+    )
+    (pin "1")
+  )
+  (symbol (lib_id "power:PWR_FLAG") (at 469.85 185.02 0) (unit 1)
+    (in_bom yes) (on_board yes)
+    (property "Reference" "FLG2" (id 0) (at 469.85 176.13 0)
+      (effects (font (size 1.27 1.27)))
+    )
+    (property "Value" "PWR_FLAG" (id 1) (at 469.85 178.67 0)
+      (effects (font (size 1.27 1.27)))
+    )
+    (property "Footprint" "" (id 2) (at 469.85 185.02 0)
+      (effects (font (size 1.27 1.27)) hide)
+    )
+    (property "Datasheet" "" (id 3) (at 469.85 185.02 0)
+      (effects (font (size 1.27 1.27)) hide)
+    )
+    (pin "1")
+  )
+  (symbol (lib_id "power:PWR_FLAG") (at 99.85 55.02 0) (unit 1)
+    (in_bom yes) (on_board yes)
+    (property "Reference" "FLG3" (id 0) (at 99.85 46.13 0)
+      (effects (font (size 1.27 1.27)))
+    )
+    (property "Value" "PWR_FLAG" (id 1) (at 99.85 48.67 0)
+      (effects (font (size 1.27 1.27)))
+    )
+    (property "Footprint" "" (id 2) (at 99.85 55.02 0)
+      (effects (font (size 1.27 1.27)) hide)
+    )
+    (property "Datasheet" "" (id 3) (at 99.85 55.02 0)
+      (effects (font (size 1.27 1.27)) hide)
+    )
+    (pin "1")
+  )
+  (symbol (lib_id "power:PWR_FLAG") (at 380.01 229.94 0) (unit 1)
+    (in_bom yes) (on_board yes)
+    (property "Reference" "FLG4" (id 0) (at 380.01 221.05 0)
+      (effects (font (size 1.27 1.27)))
+    )
+    (property "Value" "PWR_FLAG" (id 1) (at 380.01 223.59 0)
+      (effects (font (size 1.27 1.27)))
+    )
+    (property "Footprint" "" (id 2) (at 380.01 229.94 0)
+      (effects (font (size 1.27 1.27)) hide)
+    )
+    (property "Datasheet" "" (id 3) (at 380.01 229.94 0)
+      (effects (font (size 1.27 1.27)) hide)
+    )
+    (pin "1")
+  )
+  (symbol (lib_id "power:PWR_FLAG") (at 380.01 447.4 0) (unit 1)
+    (in_bom yes) (on_board yes)
+    (property "Reference" "FLG5" (id 0) (at 380.01 438.51 0)
+      (effects (font (size 1.27 1.27)))
+    )
+    (property "Value" "PWR_FLAG" (id 1) (at 380.01 441.05 0)
+      (effects (font (size 1.27 1.27)))
+    )
+    (property "Footprint" "" (id 2) (at 380.01 447.4 0)
+      (effects (font (size 1.27 1.27)) hide)
+    )
+    (property "Datasheet" "" (id 3) (at 380.01 447.4 0)
+      (effects (font (size 1.27 1.27)) hide)
+    )
+    (pin "1")
+  )
+  (symbol (lib_id "power:PWR_FLAG") (at 380.01 240.1 0) (unit 1)
+    (in_bom yes) (on_board yes)
+    (property "Reference" "FLG6" (id 0) (at 380.01 231.21 0)
+      (effects (font (size 1.27 1.27)))
+    )
+    (property "Value" "PWR_FLAG" (id 1) (at 380.01 233.75 0)
+      (effects (font (size 1.27 1.27)))
+    )
+    (property "Footprint" "" (id 2) (at 380.01 240.1 0)
+      (effects (font (size 1.27 1.27)) hide)
+    )
+    (property "Datasheet" "" (id 3) (at 380.01 240.1 0)
+      (effects (font (size 1.27 1.27)) hide)
+    )
+    (pin "1")
+  )
+  (symbol (lib_id "power:PWR_FLAG") (at 380.01 467.72 0) (unit 1)
+    (in_bom yes) (on_board yes)
+    (property "Reference" "FLG7" (id 0) (at 380.01 458.83 0)
+      (effects (font (size 1.27 1.27)))
+    )
+    (property "Value" "PWR_FLAG" (id 1) (at 380.01 461.37 0)
+      (effects (font (size 1.27 1.27)))
+    )
+    (property "Footprint" "" (id 2) (at 380.01 467.72 0)
+      (effects (font (size 1.27 1.27)) hide)
+    )
+    (property "Datasheet" "" (id 3) (at 380.01 467.72 0)
+      (effects (font (size 1.27 1.27)) hide)
+    )
+    (pin "1")
+  )
+  (symbol (lib_id "power:PWR_FLAG") (at 721.12 481.05 0) (unit 1)
+    (in_bom yes) (on_board yes)
+    (property "Reference" "FLG8" (id 0) (at 721.12 472.16 0)
+      (effects (font (size 1.27 1.27)))
+    )
+    (property "Value" "PWR_FLAG" (id 1) (at 721.12 474.7 0)
+      (effects (font (size 1.27 1.27)))
+    )
+    (property "Footprint" "" (id 2) (at 721.12 481.05 0)
+      (effects (font (size 1.27 1.27)) hide)
+    )
+    (property "Datasheet" "" (id 3) (at 721.12 481.05 0)
+      (effects (font (size 1.27 1.27)) hide)
+    )

Commit message: Mark PWR_FLAG as a real KiCad power symbol, add junctions at flag points
The previous PWR_FLAG fix (a55207f) didn't reduce ERC's violation count
-- it went from 8 to 11. My PWR_FLAG instances had a power_out-typed
pin but were built through the same generic-symbol path as the R/C/
connector stand-ins, which never sets the library symbol's own `(power)`
token. Real KiCad's power-input-pin-not-driven ERC check looks for that
token (how its own power:GND/power:PWR_FLAG etc. are authored), not just
a power_out pin sitting on an ordinary symbol -- so none of the 8 flags
actually counted as drivers, and the 3-symbol-count increase likely
added its own new findings on top.

load_generic_symbol() now sets isPower=True whenever the library
nickname is "power", and power_flag() drops an explicit junction where
each flag's wire lands on the target net's existing pin coordinate.
Verified the embedded lib_symbols copy now carries the `(power)` token,
and re-confirmed kicad-cli sch export svg/netlist still succeed and the
wire-connectivity/net-conflict check still passes.

Co-Authored-By: Claude Sonnet 5 <noreply@anthropic.com>
Claude-Session: https://claude.ai/code/session_011fHSpdvtPAVWjNqNm1QQuM
Parts:
- removed FLG1, FLG2, FLG3, FLG4, FLG5, FLG6, FLG7, FLG8: PWR_FLAG, symbol power:PWR_FLAG
Changed lines of the file:
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@@
     (comment 4 "Populated schematic: components placed & wired per verified pin maps; generic support passives are engineering defaults, not datasheet-sourced -- see kicad/README.md")
+  )
+  (junction (at 99.85 325.72) (diameter 0) (color 0 0 0 0)
+  )
+  (junction (at 469.85 193.02) (diameter 0) (color 0 0 0 0)
+  )
+  (junction (at 99.85 63.02) (diameter 0) (color 0 0 0 0)
+  )
+  (junction (at 380.01 237.94) (diameter 0) (color 0 0 0 0)
+  )
+  (junction (at 380.01 455.4) (diameter 0) (color 0 0 0 0)
+  )
+  (junction (at 380.01 248.1) (diameter 0) (color 0 0 0 0)
+  )
+  (junction (at 380.01 475.72) (diameter 0) (color 0 0 0 0)
+  )
+  (junction (at 721.12 489.05) (diameter 0) (color 0 0 0 0)
   )
   (no_connect (at 359.69 255.72))

Commit message: Fix wire-routing shorts: ERC's pin_to_pin violations were real, not power-flag noise
The real cause of ERC's 8 (then 11) violations was never the power-flag
work -- it was a routing bug in Builder.wire()'s naive 2-segment L-route.
Its first leg reused the source pin's native row/column and its second
leg the destination's; both are shared by every sibling pin in the same
stack (all of DRV8353S's top-row pins share one Y, every pin on a
component's right edge shares one X). Whenever two unrelated wires'
long traversal fell on one of those shared coordinates, KiCad correctly
read the collinear, overlapping segments as one net -- an actual short
between signals like DRV8353S's GHA/GLA/GHB gate-driver outputs, exactly
what ERC's "pin_to_pin: Output and Output are connected" reported.

wire() now gives every bent route a short, per-call-unique lead-in off
the source's native coordinate and lead-out into the destination's (kept
under the 2.54mm pin pitch, so a lead-in/out leg can't overlap an
adjacent sibling's own lead-in/out), with the long traversal run down a
row/column unique to that one wire. The two remaining straight-wire
cases this didn't cover (ADM2582E/ADM2587E's Y-A and Z-B half-duplex
ties, whose pins interleave on the same shared column so a direct tie
between one pair overlaps the other pair's span) get an explicit
jogged-out route instead.

Added a local collinear-overlap checker (union-find over labels/wires,
then pairwise range-overlap test between differently-identified nets)
since this class of bug doesn't show up in the kiutils round-trip or a
plain SVG export -- only in real connectivity analysis, which the KiCad
version available in this sandbox (7.0.11, predates `sch erc`/`pcb drc`)
can't run directly. It found 61 pre-existing conflicts on the original
routing, confirmed 0 after this fix, and independently corroborates
what CI's real KiCad-9 ERC run reported.

Co-Authored-By: Claude Sonnet 5 <noreply@anthropic.com>
Claude-Session: https://claude.ai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
Connections:
- net 3V3: no longer R2.2, U1.9 (GD_SPI_MISO), U5.27 (SDO), U5.31 (ENABLE)
- net CAN_ISO_GND: no longer BT6.2 (-), C1.2 (-), C2.1, C2.2, C3.2, C6.1, C6.2, C7.1, C7.2, C8.1, C8.2, J1.1 (Pin_1), J1.2 (Pin_2), J1.4 (Pin_4), J2.1 (Pin_1), J2.2 (Pin_2), R1.2, R10.2, R4.2, R5.2, R6.2, R8.2, SH1.1 (SHIELD_GND), SH2.1 (SHIELD_GND), U1.12 (SWDIO), U1.13 (SWCLK), U1.32 (VCORE), U1.38 (NRST), U1.41 (VSS), U1.6 (CAN_RX), U2.16 (NCI/GND), U2.2 (GND), U2.23 (GND), U2.32 (GND), U2.9 (GND), U3.1 (GND1), U3.10 (GND1), U3.13 (CANL), U3.14 (CANH), U3.16 (VISOIN), U3.2 (GND1), U3.5 (RXD), U3.6 (SILENT), U3.8 (STBY), U4.1 (GND1), U4.10 (GND1), U4.3 (GND1), U4.9 (GND1), U5.10 (SNA), U5.11 (SNB), U5.20 (SNC), U5.24 (VREF), U5.25 (AGND), U5.38 (DVDD), U5.39 (GND), U5.40 (VGLS), U6.1 (IN-), U6.2 (GND), U7.1 (IN-), U7.2 (GND), U8.1 (IN-), U8.2 (GND)
- net ISENSE_A_HI: no longer Q1.1 (G), Q2.1 (G), Q3.1 (G), Q4.1 (G), Q4.3 (S), R5.1, U5.12 (SPB), U5.13 (GLB), U5.15 (GHB), U5.6 (GHA), U5.8 (GLA), U7.8 (IN+)
- net RS485_A: no longer J3.2 (Pin_2), U4.15 (Z), U4.17 (B)
- net RS485_ISO_GND: no longer U1.1 (RS485_RXD), U4.4 (RxD)
- net VM: no longer C4.1, C4.2, C5.1, U5.1 (CPL), U5.2 (CPH), U5.5 (VCP)
- net at U1.44 (TPM_SPI_MISO), U2.24 (MISO): no longer U1.58 (TPM_PIRQ#), U2.18 (PIRQ#)
- net at Q5.1 (G), U5.16 (GHC): no longer Q6.1 (G), U5.18 (GLC)
- new net: Q4.1 (G), U5.13 (GLB)
- new net: U1.1 (RS485_RXD), U4.4 (RxD)
- new net: U1.10 (GD_SPI_SCK), U5.29 (SCLK)
- new net: U1.11 (GD_SPI_MOSI), U5.28 (SDI)
- new net: J1.1 (Pin_1), U1.12 (SWDIO)
- new net: J1.2 (Pin_2), U1.13 (SWCLK)
- new net: U1.30 (GD_SPI_CS), U5.30 (nSCS)
- new net: C2.1, U1.32 (VCORE)
- new net: U1.33 (PWM_AH), U5.32 (INHA)
- new net: U1.34 (PWM_AL), U5.33 (INLA)
- new net: U1.35 (PWM_CH), U5.36 (INHC)
- new net: R1.2, U1.38 (NRST)
- new net: U1.42 (TPM_SPI_CS), U2.20 (CS#)
- new net: U1.45 (TPM_SPI_MOSI), U2.21 (MOSI)
- new net: U1.46 (TPM_SPI_SCK), U2.19 (SCLK)
- new net: U1.47 (PWM_BH), U5.34 (INHB)
- new net: U1.48 (PWM_BL), U5.35 (INLB)
- new net: U1.51 (PWM_CL), U5.37 (INLC)
- new net: U1.58 (TPM_PIRQ#), U2.18 (PIRQ#)
- new net: U1.59 (TPM_RST#), U2.17 (RST#)
- new net: U1.6 (CAN_RX), U3.5 (RXD)
- new net: U1.9 (GD_SPI_MISO), U5.27 (SDO)
- new net: C4.2, U5.1 (CPL)
- new net: Q3.1 (G), U5.15 (GHB)
- new net: Q6.1 (G), U5.18 (GLC)
- new net: C4.1, U5.2 (CPH)
- new net: C6.1, U5.24 (VREF)
- new net: R2.2, U5.31 (ENABLE)
- new net: C7.1, U5.38 (DVDD)
- new net: C8.1, U5.40 (VGLS)
- new net: C5.1, U5.5 (VCP)
- new net: Q1.1 (G), U5.6 (GHA)
- new net: Q2.1 (G), U5.8 (GLA)
- new net: J2.2 (Pin_2), U3.13 (CANL)
- new net: J2.1 (Pin_1), U3.14 (CANH)
- new net CAN_VISOIN_OPEN: U3.16 (VISOIN)
- new net GND: BT6.2 (-), C1.2 (-), C2.2, C3.2, C6.2, C7.2, C8.2, J1.4 (Pin_4), R10.2, R4.2, R5.2, R6.2, R8.2, SH1.1 (SHIELD_GND), SH2.1 (SHIELD_GND), U1.41 (VSS), U2.16 (NCI/GND), U2.2 (GND), U2.23 (GND), U2.32 (GND), U2.9 (GND), U3.1 (GND1), U3.10 (GND1), U3.2 (GND1), U3.6 (SILENT), U3.8 (STBY), U4.1 (GND1), U4.10 (GND1), U4.3 (GND1), U4.9 (GND1), U5.10 (SNA), U5.11 (SNB), U5.20 (SNC), U5.25 (AGND), U5.39 (GND), U6.1 (IN-), U6.2 (GND), U7.1 (IN-), U7.2 (GND), U8.1 (IN-), U8.2 (GND)
- new net ISENSE_B_HI: Q4.3 (S), R5.1, U5.12 (SPB), U7.8 (IN+)
- new net RS485_B: J3.2 (Pin_2), U4.15 (Z), U4.17 (B)
