File: builds/6s/50A/CAN_485_faraday/kicad/open_secure_esc_6s_50a_can485_faraday.kicad_sch (KiCad schematic)
At the start: 44 parts, among them J1 J_SWD, J2 J_CAN, J3 J_RS485, J4 J_MOTOR, Q1 IRFB4110PBF, Q2 IRFB4110PBF, Q3 IRFB4110PBF, Q4 IRFB4110PBF, Q5 IRFB4110PBF, Q6 IRFB4110PBF, U1 MSPM0G3507SPMR, U2 SLB9672, U3 ADM3055E/ADM3057E, U4 ADM2582E/ADM2587E, U5 DRV8353S, U6 INA240, U7 INA240, U8 INA240

Commit message: Migrate MCU to NXP S32K144, drop SLB9672 TPM in favor of on-chip CSEc
Replaces the project MCU (MSPM0G3507) with the NXP S32K144, whose on-chip
CSEc (Cryptographic Services Engine, SHE-compliant) security module now
provides message authentication in place of the discrete Infineon SLB9672
TPM, which is removed from the design entirely.

- REFERENCES.md: add [31] (S32K1xx Data Sheet, local copy verified against
  CSEc, packages, memory, power-pin names, RESET_B/SWD_CLK/SWD_DIO); mark
  [1] and [2] superseded/dropped rather than repurposed, per AGENTS.md.
- symbols/specs/S32K144.json + symbols/S32K144.kicad_sym: new MCU symbol.
  Feature-level facts VERIFIED against the local datasheet; physical pin
  numbers are an UNVERIFIED PLACEHOLDER PIN MAP since the datasheet defers
  the actual pinout to the S32K1xx Reference Manual (not obtained, nxp.com
  fetch blocked this session) -- flagged per AGENTS.md SS1.3/SS3, tracked
  in TODO.md 1.11/11.7. No TPM_SPI_*/PIRQ#/RST# pins: CSEc has no external
  pins of its own, freeing the LPSPI channel the TPM used to occupy.
- Remove symbols/{MSPM0G3507,SLB9672}.kicad_sym and their specs (unused);
  keep both datasheets under docs/datasheets/ so the REFERENCES.md
  citation history stays resolvable.
- README.md, symbols/README.md, builds/6s/50A/CAN_485_faraday/README.md,
  TODO.md: update MCU/TPM lines, BOM, per-component tables, and WBS items
  (3.1, 4.1-4.4, 11.2/11.3/11.7, 12.1) to match.
- builds/6s/50A/CAN_485_faraday/kicad/: swap U1 to S32K144, drop U2
  (SLB9672) and its wiring, add VDDA/VREFH/VREFL_VSSA_VSS decoupling per
  the datasheet's "VDD and VDDA must be shorted to a common source"
  requirement, regenerate .kicad_sch/.kicad_pcb via the existing
  gen_schematic.py/gen_pcb.py tooling. Connectivity check clean,
  check_shorts.py clean, kiutils round-trip validated.
Parts:
- removed U1: MSPM0G3507SPMR, Package_QFP:LQFP-64_10x10mm_P0.5mm, symbol MSPM0G3507:MSPM0G3507
- removed U2: SLB9672, Package_DFN_QFN:QFN-32-1EP_5x5mm_P0.5mm, symbol SLB9672:SLB9672
- added U1: S32K144, Package_QFP:LQFP-64_10x10mm_P0.5mm, symbol S32K144:S32K144
- C2: Note MSPM0 VCORE decoupling, generic value per typical TI refere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 -> MCU VDD decoupling, generic value. 3V3 regulator selection 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
- C3: Note MCU VDD decoupling, generic value. 3V3 regulator selection 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 -> MCU VDDA decoupling, generic value. Datasheet [31] p.13 req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
- R1: Note Generic NRST pull-up, engineering default -- not datasheet-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 -> Generic RESET_B pull-up, engineering default -- not datashe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
Connections:
- net 3V3: now also C2.1, U1.1 (VDD), U1.3 (VDDA), U1.4 (VREFH)
- net ADC_IU: now also U1.18 (ADC_IU)
- net ADC_IV: now also U1.19 (ADC_IV)
- net ADC_IW: now also U1.20 (ADC_IW)
- net GND: now also U1.2 (VSS), U1.5 (VREFL_VSSA_VSS)
- net RS485_DE_RE: now also U1.13 (RS485_DE_RE)
- net VBUS_SENSE: now also U1.21 (ADC_VBUS)
- net at U4.4 (RxD): now also U1.12 (RS485_RXD)
- net at U5.29 (SCLK): now also U1.17 (GD_SPI_SCK)
- net at U5.28 (SDI): now also U1.16 (GD_SPI_MOSI)
- net at J1.1 (Pin_1): now also U1.8 (SWD_DIO)
- net at J1.2 (Pin_2): now also U1.7 (SWD_CLK)
- net at U5.30 (nSCS): now also U1.14 (GD_SPI_CS)
- net at U5.32 (INHA): now also U1.22 (PWM_AH)
- net at U5.33 (INLA): now also U1.23 (PWM_AL)
- net at U5.36 (INHC): now also U1.26 (PWM_CH)
- net at R1.2: now also U1.6 (RESET_B)
- net at U5.34 (INHB): now also U1.24 (PWM_BH)
- net at U5.35 (INLB): now also U1.25 (PWM_BL)
- net at U3.7 (TXD): now also U1.9 (CAN_TX)
- net at U5.37 (INLC): now also U1.27 (PWM_CL)
- net at U3.5 (RXD): now also U1.10 (CAN_RX)
- net at U4.7 (TxD): now also U1.11 (RS485_TXD)
- net at U5.27 (SDO): now also U1.15 (GD_SPI_MISO)
- no-connect marks 24 -> 8
Other:
- note added: "No external TPM: message authentication is provided by the S32K144's own on-chip CSEc security module (internal peripheral, no dedicated pins) -- see ../README.md"

Commit message: update the data
Parts:
- renumbered BT2 to BT?, BT1 to BT?, BT3 to BT?, BT6 to BT?, BT5 to BT?, BT4 to BT?, C1 to C?, C2 to C?, C4 to C?, C6 to C?, C5 to C?, C3 to C?, C8 to C?, C7 to C?, J2 to J?, J1 to J?, J3 to J?, J4 to J?, Q1 to Q?, Q4 to Q?, Q2 to Q?, Q5 to Q?, Q3 to Q?, Q6 to Q?, R4 to R?, R6 to R?, R8 to R?, R1 to R?, R9 to R?, R3 to R?, R2 to R?, R10 to R?, R5 to R?, R7 to R?, SH1 to SH?, SH2 to SH?, U1 to U?, U3 to U?, U7 to U?, U6 to U?, U8 to U?, U4 to U?, U5 to U?
