File: builds/6s/50A/CAN_485_faraday/kicad/open_secure_esc_6s_50a_can485_faraday.kicad_sch (KiCad schematic)
At the start: 43 parts

Commit message: feat(schematic): wire the OPTIGA Trust M secure element into the 6s/50A build
Places U2 (OPTIGA Trust M) and its support passives on the CAN_485_faraday
sheet and connects it to the S32K144's LPI2C, completing the secure-element
integration at the schematic level.

Circuit follows the vendor reference exactly (REFERENCES.md [45] p.12 Sec.3
Figure 2): SDA (pin 3) and SCL (pin 8) each pulled up 10k to +3V3, 100 nF VCC
decoupling, VCC on pin 10, GND on pin 1. The five NC contacts (2/4/5/6/7) carry
explicit no-connect flags because [45] p.17 Table 6 requires they be left
floating -- they must NOT be tied to a rail.

Nets added: SE_I2C_SDA, SE_I2C_SCL, SE_RST. The three matching pins were also
added to the schematic's embedded S32K144 lib_symbol (28/29/30), which had been
carrying the stale 27-pin generation, and wired out to the same global labels.
Netlist export confirms the pin-level joins: U1.28<->U2.8 (SCL),
U1.29<->U2.3 (SDA), U1.30<->U2.9 (RST), and U2.10 on the 3V3 net.

Method -- why this is a text injection and not a regeneration:
tools/gen_schematic.py rebuilds the sheet through `kiutils`, which is not
installed on this machine and cannot be installed here. Regenerating would also
be wrong on its own terms: the committed .kicad_sch has been opened and saved by
KiCad since it was last generated, so a rebuild would discard that. The pass is
therefore non-destructive -- it only appends objects and adds three pins to one
embedded lib_symbol. The script that did it is committed as
tools/inject_optiga_secure_element.py so the change is reproducible and
auditable rather than an untraceable hand edit.

Supporting fixes so the new part resolves cleanly:
- sym-lib-table: registered the OPTIGA_TRUST_M symbol library.
- fp-lib-table: created (the build had none) and registered this repo's own
  Open_Secure_ESC.pretty footprint library.
Both cleared the lib_symbol_issues / footprint_link_issues ERC warnings the
new part initially raised.

ERC (kicad-cli 9.0.2, --severity-a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
Parts:
- added C?: 100n, Capacitor_SMD:C_0805_2012Metric, symbol Device:C
- added R? (x2): 10k, Resistor_SMD:R_0805_2012Metric, symbol Device:R
- added U?: OPTIGA_TRUST_M, Open_Secure_ESC:Infineon_PG-USON-10-2-4_3x3mm_P0.5mm_EP1.7x2.5mm, symbol OPTIGA_TRUST_M:OPTIGA_TRUST_M
Connections:
- net 3V3: now also C?.1, R?.1, R?.1, U?.10 (VCC)
- net GND: now also C?.2, U?.1 (GND)
- new net SE_I2C_SCL: R?.2, U?.28 (SE_I2C_SCL), U?.8 (SCL)
- new net SE_I2C_SDA: R?.2, U?.29 (SE_I2C_SDA), U?.3 (SDA)
- new net SE_RST: U?.30 (SE_RST), U?.9 (RST)
- no-connect marks 8 -> 13
