File: builds/6s/50A/CAN_485_faraday/kicad/open_secure_esc_6s_50a_can485_faraday.kicad_sch (KiCad schematic)
At the start: 47 parts

Commit message: update
Parts:
- added C?: 10uF, Capacitor_SMD:C_0805_2012Metric, symbol Device:C
- added R?: 10k, Resistor_SMD:R_0805_2012Metric, symbol Device:R
- C?: value 100nF -> 470nF; Note MCU VDDA decoupling, generic value. Datasheet [31] p.13 req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 -> C_VCORE for U1 (MSPM0G3518-Q1). REQUIRED value: 470nF nomin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
- U?: value S32K144 -> MSPM0G3518_Q1_PM; symbol S32K144:S32K144 -> MSPM0G3518_Q1_PM:MSPM0G3518_Q1_PM; Citation [31] -> [44]
Connections:
- net 3V3: now also U?.40 (VDD), C?.1, R?.1; no longer C?.1, U?.1 (VDD), U?.3 (VDDA), U?.4 (VREFH)
- net ADC_IU: now also U?.25 (ADC_IU); no longer U?.18 (ADC_IU)
- net ADC_IV: now also U?.24 (ADC_IV); no longer U?.19 (ADC_IV)
- net ADC_IW: now also U?.26 (ADC_IW); no longer U?.20 (ADC_IW)
- net GND: now also U?.41 (VSS), C?.2; no longer U?.2 (VSS), U?.5 (VREFL_VSSA_VSS)
- net RS485_DE_RE: now also U?.37 (RS485_DE_RE); no longer U?.13 (RS485_DE_RE)
- net SE_I2C_SCL: now also U?.8 (SE_I2C_SCL); no longer U?.28 (SE_I2C_SCL)
- net SE_I2C_SDA: now also U?.9 (SE_I2C_SDA); no longer U?.29 (SE_I2C_SDA)
- net SE_RST: now also U?.7 (SE_RST); no longer U?.30 (SE_RST)
- net VBUS_SENSE: now also U?.17 (ADC_VBUS); no longer U?.21 (ADC_VBUS)
- net at U?.5 (RXD): now also U?.31 (CAN_RX); no longer U?.10 (CAN_RX)
- net at U?.7 (TxD): now also U?.33 (RS485_TXD); no longer U?.11 (RS485_TXD)
- net at U?.12 (SWDIO): now also J?.1 (Pin_1); no longer U?.4 (RxD)
- net at U?.30 (nSCS): now also U?.1 (GD_SPI_CS); no longer U?.14 (GD_SPI_CS)
- net at U?.27 (SDO): now also U?.2 (GD_SPI_MISO); no longer U?.15 (GD_SPI_MISO)
- net at U?.28 (SDI): now also U?.3 (GD_SPI_MOSI); no longer U?.16 (GD_SPI_MOSI)
- net at U?.29 (SCLK): now also U?.4 (GD_SPI_SCK); no longer U?.17 (GD_SPI_SCK)
- net at U?.32 (INHA): now also U?.54 (PWM_AH); no longer U?.22 (PWM_AH)
- net at U?.33 (INLA): now also U?.55 (PWM_AL); no longer U?.23 (PWM_AL)
- net at U?.34 (INHB): now also U?.52 (PWM_BH); no longer U?.24 (PWM_BH)
- net at U?.35 (INLB): now also U?.53 (PWM_BL); no longer U?.25 (PWM_BL)
- net at U?.36 (INHC): now also U?.47 (PWM_CH); no longer U?.26 (PWM_CH)
- net at U?.37 (INLC): now also U?.48 (PWM_CL); no longer U?.27 (PWM_CL)
- net NRST: now reaches R?.2
- net NRST: now also U?.38 (NRST), R?.2; no longer U?.6 (RESET_B)
- net at J?.2 (Pin_2): now also U?.13 (SWCLK); no longer U?.7 (SWD_CLK)
- net at U?.7 (TXD): now also U?.30 (CAN_TX); no longer U?.9 (CAN_TX)
- new net: U?.34 (RS485_RXD), U?.4 (RxD)
- new net VCORE: C?.1, U?.32 (VCORE)
Other:
- note added: "MCU U1 = TI MSPM0G3518-Q1 (PM/LQFP-64). Per-frame message authentication runs on its on-chip AES-128/256 accelerator with GCM and a 4-slot hardware keystore (REFERENCES.md [44]) -- this replaced the S32K144 CSEc, which was SHE-compliant and therefore AES-128 only. Asymmetric identity and session-key agreement remain on the OPTIGA(TM) Trust M secure element U2 (REFERENCES.md [45]); the MCU AES eng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"
- note removed: "No external TPM: message authentication is provided by the S32K144's own on-chip CSEc security module (internal peripheral, no dedicated pins) -- see ../README.md"
