File: builds/6s/50A/CAN_485_faraday/kicad/open_secure_esc_6s_50a_can485_faraday.kicad_sch (KiCad schematic)
At the start: 49 parts

Commit message: Take 6S/50A build to ERC-clean, add two decision-matrix axes, start 30x60 respin
Handoff commit. The schematic is finished and verified; PCB placement is not,
and is where the next session starts (TODO.md 12.5.j).

FOUR REAL ELECTRICAL DEFECTS FIXED (not tidying)

* Gate-driver SPI reads could never have worked. REFERENCES.md [21] gives
  DRV8353S SDO (pin 27) as type OD -- "This pin requires an external pullup
  resistor". There was none. Added R14, mirroring R11 on nFAULT.
* The board had no battery input. VM reached C1/C6/R8/U5 and three MOSFET
  drains and no connector; the old PCB had a J5 footprint with no schematic
  counterpart, i.e. two netless pads.
* Four isolated-side power flags never reached their rails -- their routes
  stopped at the right Y but at x=381.5 where the pins sit at x=380.01.
* The gate driver's exposed thermal pad had no symbol pin, so it would have
  imported as an isolated copper island under the power stage.

Schematic: 0 ERC errors (was 9). All 57 symbols annotated; 8 PWR_FLAGs made
virtual; 32 lib_symbol_mismatch warnings cleared by giving this repo ownership
of the generic R/C/connector symbols it was storing under KiCad's names.

30x60 RESPIN (TODO.md 12.5) -- schematic done, placement not

Q1-Q6 -> Toshiba TPHR8504PL [49] (SMD, enables double-sided); shield ->
WE-SHC 3670209/3671209 [51][52], saving 812 mm^2; shunts 1 -> 0.5 mOhm
(2.5 W -> 1.25 W against a 3.0 W part); J4/J5 split per terminal; J1-J4 to SMD
solder pads. All six gate nets preserved by placing the new FET symbol so its
gate pin lands on the old gate pin's exact coordinate; drains and sources
rewired with the netlist verified pin-by-pin.

The FET change reduces voltage margin from 3.97x to 1.59x over a 6S pack,
accepted by the repo owner for a 5.7x conduction-loss improvement. Bounding
the drain overshoot is open and blocks fab (12.5.n).

DECISION MATRIX: added the two axes a build cannot be instantiated without --
Motor (brushed vs brushless, which changes topology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
Parts:
- removed J?: J_MOTOR, Connector_PinHeader_2.54mm:PinHeader_1x03_P2.54mm_Vertical, symbol Connector_Generic:Conn_01x03
- added J4A: PH_A_TERM, Connector_Wire:SolderWirePad_1x01_SMD_5x10mm, symbol Open_Secure_ESC_Generic:Conn_01x01
- added J4B: PH_B_TERM, Connector_Wire:SolderWirePad_1x01_SMD_5x10mm, symbol Open_Secure_ESC_Generic:Conn_01x01
- added J4C: PH_C_TERM, Connector_Wire:SolderWirePad_1x01_SMD_5x10mm, symbol Open_Secure_ESC_Generic:Conn_01x01
- added J5A: VM_TERM, Connector_Wire:SolderWire-6sqmm_1x01_D3.5mm_OD7mm, symbol Open_Secure_ESC_Generic:Conn_01x01
- added J5B: GND_TERM, Connector_Wire:SolderWire-6sqmm_1x01_D3.5mm_OD7mm, symbol Open_Secure_ESC_Generic:Conn_01x01
- added R14: 10k, Resistor_SMD:R_0805_2012Metric, symbol Open_Secure_ESC_Generic:R
- C1: renamed from C?; footprint Capacitor_THT:CP_Radial_D10.0mm_P5.00mm -> Capacitor_SMD:C_1210_3225Metric; symbol Device:C_Polarized -> Open_Secure_ESC_Generic:C_Polarized; Note Generic bulk input cap, V>=25.2V (~2x margin -> >=50V rated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 -> Package changed from a 10 mm radial THT can to 1210 SMD 202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
- C10, C2, C3, C4, C5, C6, C7, C8, C9: renamed from C?; symbol Device:C -> Open_Secure_ESC_Generic:C
- J1: renamed from J?; footprint Connector_PinHeader_2.54mm:PinHeader_1x04_P2.54mm_Vertical -> Open_Secure_ESC:SolderPad_1x04_SMD_P2.54mm; symbol Connector_Generic:Conn_01x04 -> Open_Secure_ESC_Generic:Conn_01x04; Note (none) -> Through-hole pin header -> bare SMD solder pads 2026-08-16.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
- J2, J3: renamed from J?; footprint Connector_PinHeader_2.54mm:PinHeader_1x02_P2.54mm_Vertical -> Open_Secure_ESC:SolderPad_1x02_SMD_P2.54mm; symbol Connector_Generic:Conn_01x02 -> Open_Secure_ESC_Generic:Conn_01x02; Note (none) -> Through-hole pin header -> bare SMD solder pads 2026-08-16.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
- Q1, Q2, Q3, Q4, Q5, Q6: renamed from Q?; value IRFB4110PBF -> TPHR8504PL; footprint Package_TO_SOT_THT:TO-220-3_Vertical -> Open_Secure_ESC:Toshiba_2-5W1A_SOP-Advance-N_5.15x6.1mm_P1.27mm; symbol IRFB4110PBF:IRFB4110PBF -> TPHR8504PL:TPHR8504PL; Note (none) -> Toshiba TPHR8504PL, 40 V / 0.7 mOhm / 150 A, 2-5W1A SOP Adv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
- R1, R2, R3: renamed from R?; value 1mOhm -> 0.5mOhm; Note (none) -> Halved from 1 mOhm 2026-08-16. At the build's 50 A rating a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
- R10, R11, R12, R13, R4, R5, R6, R7, R8, R9: renamed from R?; symbol Device:R -> Open_Secure_ESC_Generic:R
- SH1: renamed from SH?; value WE-SHC 3670375 (frame) -> WE-SHC 3670209 (frame); footprint (none) -> Open_Secure_ESC:Wurth_WE-SHC_3670209_Frame_15.3x20.9mm; symbol WE_SHC_3670375:WE_SHC_3670375 -> WE_SHC_3670209:WE_SHC_3670209
- SH2: renamed from SH?; value WE-SHC 3671375 (cover) -> WE-SHC 3671209 (cover); symbol WE_SHC_3671375:WE_SHC_3671375 -> WE_SHC_3671209:WE_SHC_3671209
- U5: renamed from U?; footprint (none) -> Open_Secure_ESC:TI_RTA0040B_WQFN-40_6x6mm_P0.5mm_EP4.15x4.15mm
- gave numbers to parts that had none: 13
Connections:
- net 3V3: now also R14.1
- net GND: now also U5.41 (PAD), J5B.1 (Pin_1)
- net ISENSE_A_HI: now also Q2.1 (S), Q2.2 (S)
- net ISENSE_B_HI: now also Q4.1 (S), Q4.2 (S)
- net ISENSE_C_HI: now also Q6.1 (S), Q6.2 (S)
- net PH_A: now also Q1.1 (S), Q1.2 (S), Q2.5 (D), Q2.6 (D), Q2.7 (D), Q2.8 (D), J4A.1 (Pin_1); no longer Q2.2 (D)
- net PH_B: now also Q3.1 (S), Q3.2 (S), Q4.5 (D), Q4.6 (D), Q4.7 (D), Q4.8 (D), J4B.1 (Pin_1); no longer Q4.2 (D)
- net PH_C: now also Q5.1 (S), Q5.2 (S), Q6.5 (D), Q6.6 (D), Q6.7 (D), Q6.8 (D), J4C.1 (Pin_1); no longer Q6.2 (D)
- net VM: now also Q1.5 (D), Q1.6 (D), Q1.7 (D), Q1.8 (D), Q3.5 (D), Q3.6 (D), Q3.7 (D), Q3.8 (D), Q5.5 (D), Q5.6 (D), Q5.7 (D), Q5.8 (D), J5A.1 (Pin_1); no longer Q1.2 (D), Q3.2 (D), Q5.2 (D)
- net at U5.6 (GHA): now also Q1.4 (G); no longer Q1.1 (G)
- net GD_SPI_MISO: now reaches U1.2 (GD_SPI_MISO), U5.27 (SDO)
- net GD_SPI_MISO: now also R14.2
- net at U5.13 (GLB): now also Q4.4 (G); no longer Q4.1 (G)
- net at U5.8 (GLA): now also Q2.4 (G); no longer Q2.1 (G)
- net at U5.16 (GHC): now also Q5.4 (G); no longer Q5.1 (G)
- net at U5.15 (GHB): now also Q3.4 (G); no longer Q3.1 (G)
- net at U5.18 (GLC): now also Q6.4 (G); no longer Q6.1 (G)

Commit message: Fit the isolated-supply ferrites -- which fixes a supply that was never wired
Asked to integrate the Murata bead the repo owner supplied. Reading the two
isolator pin tables first turned this from an EMC improvement into a defect
fix: the isolated side of BOTH transceivers was unwired.

    CAN_VISOOUT        U3.19 only          dangling
    CAN_VISOIN_OPEN    U3.16 only          dangling
    CAN_ISO_GND        U3.11,12,15,18,20   all merged
    RS485_VISOOUT      U4.12 only          dangling
    RS485_VISOIN_OPEN  U4.19 only          dangling
    RS485_ISO_GND      U4.11,14,16,20      all merged

[10] p.15: "Connect this pin through a ferrite bead and short the PCB trace to
VISOIN FOR OPERATION." [9] p.8: "This pin must be connected externally to
VISOIN." That connection did not exist, so neither bus side had a supply.

Both parts also require the isolated grounds SPLIT, not merged. [10] pins
18,20 GNDISO: "Connect these pins together through one ferrite bead to PCB
ground (bus side)." [9] pins 11,14: "It is recommended to connect Pin 11 and
Pin 14 together through one ferrite bead to PCB ground." And [9] pin 16:
"Ground, Bus Side. DO NOT CONNECT THIS PIN TO PIN 14 AND PIN 11." The
pre-existing net merged exactly the pins that sentence forbids merging.

Four BLM15HD182SN1D fitted -- 1800 ohm at 100 MHz / 2700 ohm at 1 GHz, which
meets [9] p.17's "approximately 2 kohm between the 100 MHz and 1 GHz frequency
range", and is the part [10] Table 12 names by number for this role. Current
rating checked rather than assumed: 200 mA / 2.2 ohm max DCR against
isolated-side transceiver current only, and [9] Table 14 confirms the ADM2582E
has "no current available externally on VISOOUT".

  ERC  0 errors; CAN_VISOOUT and RS485_VISOOUT no longer dangle
  DRC  0 electrical violations

CORRECTION TO THE PREVIOUS COMMIT: it said the ADM3055E "states the reverse
for itself" on ferrites, so the gap was "specifically U4". Wrong. [10] p.25
asks for them just as plainly -- "filter both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
Parts:
- added FB1, FB2, FB3, FB4: BLM15HD182SN1D, Inductor_SMD:L_0402_1005Metric, symbol BLM15HD182SN1D:BLM15HD182SN1D
Connections:
- net CAN_ISO_GND: now also FB2.2; no longer U3.18 (GNDISO), U3.20 (GNDISO)
- net CAN_VISOOUT: now also FB1.1
- net RS485_ISO_GND: now also FB4.2; no longer U4.11 (GND2), U4.14 (GND2)
- net RS485_VISOOUT: now also FB3.1
- net CAN_VISOIN_OPEN renamed CAN_VISOIN
- net CAN_VISOIN: now also FB1.2
- net RS485_VISOIN_OPEN renamed RS485_VISOIN
- net RS485_VISOIN: now also FB3.2
- new net CAN_GNDISO: FB2.1, U3.18 (GNDISO), U3.20 (GNDISO)
- new net RS485_GNDISO: FB4.1, U4.11 (GND2), U4.14 (GND2)
Changed lines of the file:
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@@
     (stroke (width 0) (type default))
   )
+  (wire (pts (xy 539.85 788.89) (xy 539.85 793.9699999999999))
+    (stroke (width 0.0))
+  )
+  (wire (pts (xy 579.85 788.89) (xy 579.85 793.9699999999999))
+    (stroke (width 0.0))
+  )
   (text "nFAULT: pulled up only, not wired to MCU in this build -- open item, see ../README.md"
     (at 629.85 502.54 0)
@@
     )
   )
-  (global_label "CAN_VISOIN_OPEN" (shape passive) (at 385.09 211.27 0)
+  (global_label "CAN_VISOIN" (shape passive) (at 385.09 211.27 0)
     (effects (font (size 1.27 1.27)))
     (property "Intersheetrefs" "${INTERSHEET_REFS}" (at 385.09 211.27 0)
@@
     )
   )
-  (global_label "CAN_ISO_GND" (shape passive) (at 385.09 221.43 0)
+  (global_label "CAN_GNDISO" (shape passive) (at 385.09 221.43 0)
     (effects (font (size 1.27 1.27)))
     (property "Intersheetrefs" "${INTERSHEET_REFS}" (at 385.09 221.43 0)
@@
     )
   )
-  (global_label "RS485_ISO_GND" (shape passive) (at 385.09 418.57 0)
+  (global_label "RS485_GNDISO" (shape passive) (at 385.09 418.57 0)
     (effects (font (size 1.27 1.27)))
     (property "Intersheetrefs" "${INTERSHEET_REFS}" (at 385.09 418.57 0)
@@
     )
   )
-  (global_label "RS485_ISO_GND" (shape passive) (at 385.09 426.19 0)
+  (global_label "RS485_GNDISO" (shape passive) (at 385.09 426.19 0)
     (effects (font (size 1.27 1.27)))
     (property "Intersheetrefs" "${INTERSHEET_REFS}" (at 385.09 426.19 0)
@@
     )
   )
-  (global_label "RS485_VISOIN_OPEN" (shape passive) (at 385.09 438.89 0)
+  (global_label "RS485_VISOIN" (shape passive) (at 385.09 438.89 0)
     (effects (font (size 1.27 1.27)))
     (property "Intersheetrefs" "${INTERSHEET_REFS}" (at 385.09 438.89 0)
@@
     )
   )
-  (global_label "CAN_ISO_GND" (shape passive) (at 385.09 216.35 0)
+  (global_label "CAN_GNDISO" (shape passive) (at 385.09 216.35 0)
     (effects (font (size 1.27 1.27)))
     (property "Intersheetrefs" "${INTERSHEET_REFS}" (at 385.09 216.35 0)
@@
     )
   )
-  (global_label "CAN_VISOIN_OPEN" (shape passive) (at 419.85 793.97 270)
+  (global_label "CAN_VISOIN" (shape passive) (at 419.85 793.97 270)
     (effects (font (size 1.27 1.27)) (justify left))
     (property "Intersheetrefs" "${INTERSHEET_REFS}" (at 419.85 793.97 0)
@@
     )
   )
-  (global_label "RS485_VISOIN_OPEN" (shape passive) (at 459.85 793.97 270)
+  (global_label "RS485_VISOIN" (shape passive) (at 459.85 793.97 270)
     (effects (font (size 1.27 1.27)) (justify left))
     (property "Intersheetrefs" "${INTERSHEET_REFS}" (at 459.85 793.97 0)
@@
     )
   )
+  (global_label "CAN_VISOOUT" (shape input) (at 422.38 200.0 180)
+    (effects (font (size 1.27 1.27)))
+  )
+  (global_label "CAN_VISOIN" (shape input) (at 437.62 200.0 0)
+    (effects (font (size 1.27 1.27)))
+  )
+  (global_label "CAN_GNDISO" (shape input) (at 422.38 215.0 180)
+    (effects (font (size 1.27 1.27)))
+  )
+  (global_label "CAN_ISO_GND" (shape input) (at 437.62 215.0 0)
+    (effects (font (size 1.27 1.27)))
+  )
+  (global_label "RS485_VISOOUT" (shape input) (at 422.38 420.0 180)
+    (effects (font (size 1.27 1.27)))
+  )
+  (global_label "RS485_VISOIN" (shape input) (at 437.62 420.0 0)
+    (effects (font (size 1.27 1.27)))
+  )
+  (global_label "RS485_GNDISO" (shape input) (at 422.38 435.0 180)
+    (effects (font (size 1.27 1.27)))
+  )
+  (global_label "RS485_ISO_GND" (shape input) (at 437.62 435.0 0)
+    (effects (font (size 1.27 1.27)))
+  )
+  (global_label "CAN_GNDISO" (shape input) (at 539.85 793.9699999999999 270)
+    (effects (font (size 1.27 1.27)))
+  )
+  (global_label "RS485_GNDISO" (shape input) (at 579.85 793.9699999999999 270)
+    (effects (font (size 1.27 1.27)))
+  )
   (symbol (lib_id "Open_Secure_ESC_Generic:PWR_FLAG") (at 379.85 782.54 0) (unit 1)
     (in_bom no) (on_board no) (dnp no)
@@
         )
       )
+    )
+  )
+  (symbol (lib_id "BLM15HD182SN1D:BLM15HD182SN1D") (at 430.0 200.0 0) (unit 1)
+    (in_bom yes) (on_board yes)
+    (property "Reference" "FB1" (at 430.0 196.19 0)
+      (effects (font (size 1.27 1.27)))
+    )
+    (property "Value" "BLM15HD182SN1D" (at 430.0 203.81 0)
+      (effects (font (size 1.27 1.27)))
+    )
+    (property "Footprint" "Inductor_SMD:L_0402_1005Metric" (at 430.0 200.0 0)
+      (effects (font (size 1.27 1.27)) hide)
+    )
+    (property "Datasheet" "docs/datasheets/ENFA0024.pdf" (at 430.0 200.0 0)
+      (effects (font (size 1.27 1.27)) hide)
+    )
+    (instances
+      (project "open_secure_esc_6s_50a_can485_faraday"
+        (path "/b6909b5a-de2d-4466-bb5d-8520126b59da"
+          (reference "FB1") (unit 1)
+        )
+      )
+    )
+  )
+  (symbol (lib_id "BLM15HD182SN1D:BLM15HD182SN1D") (at 430.0 215.0 0) (unit 1)
+    (in_bom yes) (on_board yes)
+    (property "Reference" "FB2" (at 430.0 211.19 0)
+      (effects (font (size 1.27 1.27)))
+    )
+    (property "Value" "BLM15HD182SN1D" (at 430.0 218.81 0)
+      (effects (font (size 1.27 1.27)))
+    )
+    (property "Footprint" "Inductor_SMD:L_0402_1005Metric" (at 430.0 215.0 0)
+      (effects (font (size 1.27 1.27)) hide)
+    )
+    (property "Datasheet" "docs/datasheets/ENFA0024.pdf" (at 430.0 215.0 0)
+      (effects (font (size 1.27 1.27)) hide)
+    )
+    (instances
+      (project "open_secure_esc_6s_50a_can485_faraday"
+        (path "/b6909b5a-de2d-4466-bb5d-8520126b59da"
+          (reference "FB2") (unit 1)
+        )
+      )
+    )
+  )
+  (symbol (lib_id "BLM15HD182SN1D:BLM15HD182SN1D") (at 430.0 420.0 0) (unit 1)
+    (in_bom yes) (on_board yes)
+    (property "Reference" "FB3" (at 430.0 416.19 0)
+      (effects (font (size 1.27 1.27)))
+    )
+    (property "Value" "BLM15HD182SN1D" (at 430.0 423.81 0)
+      (effects (font (size 1.27 1.27)))
+    )
+    (property "Footprint" "Inductor_SMD:L_0402_1005Metric" (at 430.0 420.0 0)
+      (effects (font (size 1.27 1.27)) hide)
+    )
+    (property "Datasheet" "docs/datasheets/ENFA0024.pdf" (at 430.0 420.0 0)
+      (effects (font (size 1.27 1.27)) hide)
+    )
+    (instances
+      (project "open_secure_esc_6s_50a_can485_faraday"
+        (path "/b6909b5a-de2d-4466-bb5d-8520126b59da"
+          (reference "FB3") (unit 1)
+        )
+      )
+    )
+  )
+  (symbol (lib_id "BLM15HD182SN1D:BLM15HD182SN1D") (at 430.0 435.0 0) (unit 1)
+    (in_bom yes) (on_board yes)
+    (property "Reference" "FB4" (at 430.0 431.19 0)
+      (effects (font (size 1.27 1.27)))
+    )
+    (property "Value" "BLM15HD182SN1D" (at 430.0 438.81 0)
+      (effects (font (size 1.27 1.27)))
+    )
+    (property "Footprint" "Inductor_SMD:L_0402_1005Metric" (at 430.0 435.0 0)
+      (effects (font (size 1.27 1.27)) hide)
+    )
+    (property "Datasheet" "docs/datasheets/ENFA0024.pdf" (at 430.0 435.0 0)
+      (effects (font (size 1.27 1.27)) hide)
+    )
+    (instances
+      (project "open_secure_esc_6s_50a_can485_faraday"
+        (path "/b6909b5a-de2d-4466-bb5d-8520126b59da"
+          (reference "FB4") (unit 1)
+        )
+      )
+    )
+  )
+  (symbol (lib_id "Open_Secure_ESC_Generic:PWR_FLAG") (at 539.85 782.54 0) (unit 1)
+    (in_bom no) (on_board no)
+    (property "Reference" "#FLG0" (at 539.85 782.54 0)
+      (effects (font (size 1.27 1.27)) hide)
+    )
+    (property "Value" "PWR_FLAG" (at 539.85 780.0 0)
+      (effects (font (size 1.27 1.27)))
+    )
+    (instances
+      (project "open_secure_esc_6s_50a_can485_faraday"
+        (path "/b6909b5a-de2d-4466-bb5d-8520126b59da"
+          (reference "#FLG0") (unit 1)
+        )
+      )
+    )
+  )
+  (symbol (lib_id "Open_Secure_ESC_Generic:PWR_FLAG") (at 579.85 782.54 0) (unit 1)
+    (in_bom no) (on_board no)
+    (property "Reference" "#FLG0" (at 579.85 782.54 0)
+      (effects (font (size 1.27 1.27)) hide)
+    )
+    (property "Value" "PWR_FLAG" (at 579.85 780.0 0)
+      (effects (font (size 1.27 1.27)))
+    )
+    (instances
+      (project "open_secure_esc_6s_50a_can485_faraday"
+        (path "/b6909b5a-de2d-4466-bb5d-8520126b59da"
+          (reference "#FLG0") (unit 1)
+        )
+      )

Commit message: Add the eight isolated-supply capacitors; stage all twelve parts off-board
The repo owner asked for the remaining isolated-side components to be put
beside the board for hand placement. Done, and the four ferrites from the
previous commit moved out to join them -- the whole group stages together.

    FB1-FB4   staging column at x = 32 mm
    C11-C18   staging column at x = 40 mm
    board outline ends at x = 25.45 mm

Capacitor values and pin pairings are quoted from the datasheets, not chosen:

  [10] p.15 pin 19 VISOOUT : "requires 0.22uF and 10uF capacitors to GNDISO"
  [10] p.15 pin 16 VISOIN  : "requires 0.01uF and 0.1uF decoupling capacitors"
  [9]  p.17                : "0.1 uF and 10 uF for VISOOUT at Pin 11 and Pin
                              12 ... 0.01 uF and 0.1 uF ... for VISOIN at Pin
                              19 and Pin 20"

The two isolated grounds are deliberately not interchangeable: VISOOUT
reservoirs return to the dc-to-dc converter ground (CAN_GNDISO /
RS485_GNDISO), VISOIN decouplers to the bus-side ground (CAN_ISO_GND /
RS485_ISO_GND), and the beads bridge them. Final net topology:

  CAN_VISOOUT    C11.1 C12.1 FB1.1 U3.19
  CAN_GNDISO     C11.2 C12.2 FB2.1 U3.18 U3.20
  CAN_VISOIN     C13.1 C14.1 FB1.2 U3.16
  CAN_ISO_GND    C13.2 C14.2 FB2.2 U3.11 U3.12 U3.15
  RS485_VISOOUT  C15.1 C16.1 FB3.1 U4.12
  RS485_GNDISO   C15.2 C16.2 FB4.1 U4.11 U4.14
  RS485_VISOIN   C17.1 C18.1 FB3.2 U4.19
  RS485_ISO_GND  C17.2 C18.2 FB4.2 U4.16 U4.20

ERC 0 errors. DRC 0 electrical violations. Remaining DRC is 45 silkscreen,
12 drill (12.5.x), 10 starved_thermal on GND.

Package (0805) and voltage rating are AGENTS.md Sec.4 engineering defaults
matching C2..C10. No MPN is claimed for the capacitors -- none has been
selected, and inventing one would be a fabricated citation.

A geometry mistake made and fixed here: the capacitors were first given
horizontal labels at (x +/- 7.62, y), copying the two-terminal R and ferrite
symbols. The generic C symbol is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
Parts:
- added C11, C15: 10uF, Capacitor_SMD:C_0805_2012Metric, symbol Open_Secure_ESC_Generic:C
- added C12: 220nF, Capacitor_SMD:C_0805_2012Metric, symbol Open_Secure_ESC_Generic:C
- added C13, C16, C17: 100nF, Capacitor_SMD:C_0805_2012Metric, symbol Open_Secure_ESC_Generic:C
- added C14, C18: 10nF, Capacitor_SMD:C_0805_2012Metric, symbol Open_Secure_ESC_Generic:C
Connections:
- net CAN_GNDISO: now also C11.2, C12.2
- net CAN_ISO_GND: now also C13.2, C14.2
- net CAN_VISOIN: now also C13.1, C14.1
- net CAN_VISOOUT: now also C11.1, C12.1
- net RS485_GNDISO: now also C15.2, C16.2
- net RS485_ISO_GND: now also C17.2, C18.2
- net RS485_VISOIN: now also C17.1, C18.1
- net RS485_VISOOUT: now also C15.1, C16.1
