File: builds/6s/50A/CAN_485_faraday/kicad/open_secure_esc_6s_50a_can485_faraday.kicad_pcb (KiCad board)
At the start: 4 copper layers, 25.4 x 60.1 mm, 47 parts, among them J1 SolderPad_1x04_SMD_P2.54mm, J2 SolderPad_1x02_SMD_P2.54mm, J3 SolderPad_1x02_SMD_P2.54mm, J4A SolderWirePad_1x01_SMD_5x10mm, J4B SolderWirePad_1x01_SMD_5x10mm, J4C SolderWirePad_1x01_SMD_5x10mm, J5A SolderWire-6sqmm_1x01_D3.5mm_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, J5B SolderWire-6sqmm_1x01_D3.5mm_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, Q1 Toshiba_2-5W1A_SOP-Advance-N_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, Q2 Toshiba_2-5W1A_SOP-Advance-N_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, Q3 Toshiba_2-5W1A_SOP-Advance-N_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, Q4 Toshiba_2-5W1A_SOP-Advance-N_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, Q5 Toshiba_2-5W1A_SOP-Advance-N_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, Q6 Toshiba_2-5W1A_SOP-Advance-N_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, U1 LQFP-64_10x10mm_P0.5mm, U2 Infineon_PG-USON-10-2-4_3x3mm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, U3 SOIC-20W_7.5x12.8mm_P1.27mm, U4 SOIC-20W_7.5x12.8mm_P1.27mm, U5 TI_RTA0040B_WQFN-40_6x6mm_P0.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, U6 SOIC-8_3.9x4.9mm_P1.27mm, U7 SOIC-8_3.9x4.9mm_P1.27mm, U8 SOIC-8_3.9x4.9mm_P1.27mm

Commit message: Read the isolator datasheets: the keepout is backwards, and creepage fails
The repo owner rotated U3 by 180 deg, which closes 12.5.aa -- U3's isolated
row now sits at x 11.28 facing J2, so the CAN runs are 0.05 and 2.59 mm
instead of 9.35 and 11.89. U4/J3 was already correct.

That left "what do we do about the keepout". Rather than guess, went to the
primary sources already in docs/datasheets/.

THE FULL-WIDTH 4-LAYER KEEPOUT IS NOT WHAT ANALOG DEVICES ASKS FOR. [9] p.17,
for a four layer board, asks for the OPPOSITE: "place an embedded stitching
capacitor between GND1 and GND2 using internal layers of the PCB planes ...
This capacitor provides a return path for high frequency common-mode noise
currents across the isolation gap." The only keepout [9] specifies is narrow
and conditional -- no GND2 (isolated) fill below the L1/L2 ferrites. So the
existing rectangle removes the very plane overlap the datasheet wants, and
the constraint that actually binds the barrier is creepage, not plane cuts.

CREEPAGE CURRENTLY FAILS. [9] Table 6 p.5 requires 7.5 mm external clearance
AND 7.5 mm creepage, input terminals to output terminals, with an explicit
footnote that pad layout must maintain it. Measured on the new placement:

    U4.11 (isolated) <-> U2.10    3.49 mm
    U4.11 (isolated) <-> U2.9     3.97 mm
    U4.11 (isolated) <-> U1.1     4.58 mm

The board undercuts the transceiver's own 5 kV rating by 4.01 mm. U1 (MCU)
and U2 (OPTIGA) sit too close to U4's isolated row. Placement call.

THE RECOMMENDED FERRITES ARE MISSING ENTIRELY. [9] p.17 instructs filtering
both GND2 pins and VISOOUT with series surface-mount ferrite beads (~2 kOhm
over 100 MHz-1 GHz) against the 180 MHz primary and 360 MHz secondary
switching harmonics. This board has no ferrites at all -- its only reference
designators are J, U, R, Q, C, SH. Schematic/BOM gap, and it bears directly
on the Faraday EMI tier. The ADM3055E says the reverse for itself ([10] p.25,
"Neither PCB stitching capacitance nor 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
Parts:
- moved C1 40.8 mm to (27.5, 67.0)
- moved R1 4.00 mm to (24.5, 63.0)
- moved Q1 3.50 mm to (24.0, 49.0)
- moved Q2 3.50 mm to (24.0, 57.0)
- moved R2 0.51 mm to (32.5, 60.5)
- turned U3 to 0 degrees
Changed lines of the file:
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@@
 	(footprint "R_2512_6332Metric"
 		(layer "F.Cu")
-		(at 24.4 67)
+		(at 24.5 63)
 		(descr "Resistor SMD 2512 (6332 Metric), square (rectangular) end terminal, IPC-7351 nominal, (Body size source: IPC-SM-782 page 72, https://www.pcb-3d.com/wordpress/wp-content/uploads/ipc-sm-782a_amendment_1_and_2.pdf), generated with kicad-footprint-generator")
 		(tags "resistor")
@@
 	(footprint "Toshiba_2-5W1A_SOP-Advance-N_5.15x6.1mm_P1.27mm"
 		(layer "F.Cu")
-		(at 24 60.5)
+		(at 24 57)
 		(descr "Toshiba 2-5W1A SOP Advance(N), 8 lead, 1.27 mm pitch, 5.15x6.10 mm package. Land pattern is TOSHIBA'S OWN, from REFERENCES.md [50] (MOSFET Product Catalog ALQ00024) p.46 -- 4.7 mm wide, castellated 4.7x4.8 mm drain land, 0.85x1.45 mm lead pads, 0.7 mm gap. Pads 1/2/3 source, 4 gate, 5-8 drain; the drain land carries the same numbers as the drain leads so they merge onto one net. NOT interchangeable with the 2-5Q1S SOP Advance variant. Generated by symbols/tools/gen_tphr8504pl_footprint.py")
 		(tags "Toshiba 2-5W1A SOP Advance N MOSFET TPHR8504PL power 5x6")
@@
 	(footprint "Toshiba_2-5W1A_SOP-Advance-N_5.15x6.1mm_P1.27mm"
 		(layer "F.Cu")
-		(at 24 52.5)
+		(at 24 49)
 		(descr "Toshiba 2-5W1A SOP Advance(N), 8 lead, 1.27 mm pitch, 5.15x6.10 mm package. Land pattern is TOSHIBA'S OWN, from REFERENCES.md [50] (MOSFET Product Catalog ALQ00024) p.46 -- 4.7 mm wide, castellated 4.7x4.8 mm drain land, 0.85x1.45 mm lead pads, 0.7 mm gap. Pads 1/2/3 source, 4 gate, 5-8 drain; the drain land carries the same numbers as the drain leads so they merge onto one net. NOT interchangeable with the 2-5Q1S SOP Advance variant. Generated by symbols/tools/gen_tphr8504pl_footprint.py")
 		(tags "Toshiba 2-5W1A SOP Advance N MOSFET TPHR8504PL power 5x6")
@@
 	(footprint "R_2512_6332Metric"
 		(layer "F.Cu")
-		(at 32.6 61)
+		(at 32.5 60.5)
 		(descr "Resistor SMD 2512 (6332 Metric), square (rectangular) end terminal, IPC-7351 nominal, (Body size source: IPC-SM-782 page 72, https://www.pcb-3d.com/wordpress/wp-content/uploads/ipc-sm-782a_amendment_1_and_2.pdf), generated with kicad-footprint-generator")
 		(tags "resistor")
@@
 	(footprint "C_1210_3225Metric"
 		(layer "F.Cu")
-		(at 32.5 26.5)
+		(at 27.5 67)
 		(descr "Capacitor SMD 1210 (3225 Metric), square (rectangular) end terminal, IPC-7351 nominal, (Body size source: IPC-SM-782 page 76, https://www.pcb-3d.com/wordpress/wp-content/uploads/ipc-sm-782a_amendment_1_and_2.pdf), generated with kicad-footprint-generator")
 		(tags "capacitor")
@@
 	(footprint "SOIC-20W_7.5x12.8mm_P1.27mm"
 		(layer "B.Cu")
-		(at 26.53 36 180)
+		(at 26.53 36)
 		(descr "SOIC, 20 Pin (JEDEC MS-013AC, https://www.analog.com/media/en/package-pcb-resources/package/233848rw_20.pdf), generated with kicad-footprint-generator ipc_gullwing_generator.py")
 		(tags "SOIC SO")
@@
 		(attr smd)
 		(fp_line
-			(start 3.86 6.51)
-			(end 3.86 6.275)
+			(start -3.86 -6.51)
+			(end -3.86 -6.275)
 			(stroke
 				(width 0.12)
@@
 		)
 		(fp_line
-			(start 3.86 -6.51)
-			(end 3.86 -6.275)
+			(start -3.86 6.51)
+			(end -3.86 6.275)
 			(stroke
 				(width 0.12)
@@
 		)
 		(fp_line
-			(start 0 6.51)
-			(end 3.86 6.51)
+			(start 0 -6.51)
+			(end -3.86 -6.51)
 			(stroke
 				(width 0.12)
@@
 		)
 		(fp_line
-			(start 0 6.51)
-			(end -3.86 6.51)
+			(start 0 -6.51)
+			(end 3.86 -6.51)
 			(stroke
 				(width 0.12)
@@
 		)
 		(fp_line
-			(start 0 -6.51)
-			(end 3.86 -6.51)
+			(start 0 6.51)
+			(end -3.86 6.51)
 			(stroke
 				(width 0.12)
@@
 		)
 		(fp_line
-			(start 0 -6.51)
-			(end -3.86 -6.51)
+			(start 0 6.51)
+			(end 3.86 6.51)
 			(stroke
 				(width 0.12)
@@
 		)
 		(fp_line
-			(start -3.86 6.51)
-			(end -3.86 6.275)
+			(start 3.86 -6.51)
+			(end 3.86 -6.275)
 			(stroke
 				(width 0.12)
@@
 		)
 		(fp_line
-			(start -3.86 -6.51)
-			(end -3.86 -6.275)
+			(start 3.86 6.51)
+			(end 3.86 6.275)
 			(stroke
 				(width 0.12)
@@
 		)
 		(fp_line
-			(start 5.93 6.27)
-			(end 5.93 -6.27)
+			(start -5.93 -6.27)
+			(end -5.93 6.27)
 			(stroke
 				(width 0.05)
@@
 		)
 		(fp_line
-			(start 5.93 -6.27)
-			(end 4 -6.27)
+			(start -5.93 6.27)
+			(end -4 6.27)
 			(stroke
 				(width 0.05)
@@
 		)
 		(fp_line
-			(start 4 6.65)
-			(end 4 6.27)
+			(start -4 -6.65)
+			(end -4 -6.27)
 			(stroke
 				(width 0.05)
@@
 		)
 		(fp_line
-			(start 4 6.27)
-			(end 5.93 6.27)
+			(start -4 -6.27)
+			(end -5.93 -6.27)
 			(stroke
 				(width 0.05)
@@
 		)
 		(fp_line
-			(start 4 -6.27)
-			(end 4 -6.65)
+			(start -4 6.27)
+			(end -4 6.65)
 			(stroke
 				(width 0.05)
@@
 		)
 		(fp_line
-			(start 4 -6.65)
-			(end -4 -6.65)
+			(start -4 6.65)
+			(end 4 6.65)
 			(stroke
 				(width 0.05)
@@
 		)
 		(fp_line
-			(start -4 6.65)
-			(end 4 6.65)
+			(start 4 -6.65)
+			(end -4 -6.65)
 			(stroke
 				(width 0.05)
@@
 		)
 		(fp_line
-			(start -4 6.27)
-			(end -4 6.65)
+			(start 4 -6.27)
+			(end 4 -6.65)
 			(stroke
 				(width 0.05)
@@
 		)
 		(fp_line
-			(start -4 -6.27)
-			(end -5.93 -6.27)
+			(start 4 6.27)
+			(end 5.93 6.27)
 			(stroke
 				(width 0.05)
@@
 		)
 		(fp_line
-			(start -4 -6.65)
-			(end -4 -6.27)
+			(start 4 6.65)
+			(end 4 6.27)
 			(stroke
 				(width 0.05)
@@
 		)
 		(fp_line
-			(start -5.93 6.27)
-			(end -4 6.27)
+			(start 5.93 -6.27)
+			(end 4 -6.27)
 			(stroke
 				(width 0.05)
@@
 		)
 		(fp_line
-			(start -5.93 -6.27)
-			(end -5.93 6.27)
+			(start 5.93 6.27)
+			(end 5.93 -6.27)
 			(stroke
 				(width 0.05)
@@
 		)
 		(fp_line
-			(start 3.75 6.4)
-			(end 3.75 -6.4)
+			(start -3.75 -6.4)
+			(end -3.75 5.4)
 			(stroke
 				(width 0.1)
@@
 		)
 		(fp_line
-			(start 3.75 -6.4)
-			(end -3.75 -6.4)
+			(start -3.75 5.4)
+			(end -2.75 6.4)
 			(stroke
 				(width 0.1)
@@
 		)
 		(fp_line
-			(start -3.75 5.4)
-			(end -2.75 6.4)
+			(start 3.75 -6.4)
+			(end -3.75 -6.4)
 			(stroke
 				(width 0.1)
@@
 		)
 		(fp_line
-			(start -3.75 -6.4)
-			(end -3.75 5.4)
+			(start 3.75 6.4)
+			(end 3.75 -6.4)
 			(stroke
 				(width 0.1)
@@
 		)
 		(pad "1" smd roundrect
-			(at -4.65 5.715 180)
+			(at -4.65 5.715)
 			(size 2.05 0.6)
 			(layers "B.Cu" "B.Mask" "B.Paste")
@@
 		)
 		(pad "2" smd roundrect
-			(at -4.65 4.445 180)
+			(at -4.65 4.445)
 			(size 2.05 0.6)
 			(layers "B.Cu" "B.Mask" "B.Paste")
@@
 		)
 		(pad "3" smd roundrect
-			(at -4.65 3.175 180)
+			(at -4.65 3.175)
 			(size 2.05 0.6)
 			(layers "B.Cu" "B.Mask" "B.Paste")
@@
 		)
 		(pad "4" smd roundrect
-			(at -4.65 1.905 180)
+			(at -4.65 1.905)
 			(size 2.05 0.6)
 			(layers "B.Cu" "B.Mask" "B.Paste")
@@
 		)
 		(pad "5" smd roundrect
-			(at -4.65 0.635 180)
+			(at -4.65 0.635)
 			(size 2.05 0.6)
 			(layers "B.Cu" "B.Mask" "B.Paste")
@@
 		)
 		(pad "6" smd roundrect
-			(at -4.65 -0.635 180)
+			(at -4.65 -0.635)
 			(size 2.05 0.6)
 			(layers "B.Cu" "B.Mask" "B.Paste")
@@
 		)
 		(pad "7" smd roundrect
-			(at -4.65 -1.905 180)
+			(at -4.65 -1.905)
 			(size 2.05 0.6)
 			(layers "B.Cu" "B.Mask" "B.Paste")
@@
 		)
 		(pad "8" smd roundrect
-			(at -4.65 -3.175 180)
+			(at -4.65 -3.175)
 			(size 2.05 0.6)
 			(layers "B.Cu" "B.Mask" "B.Paste")
@@
 		)
 		(pad "9" smd roundrect
-			(at -4.65 -4.445 180)
+			(at -4.65 -4.445)
 			(size 2.05 0.6)
 			(layers "B.Cu" "B.Mask" "B.Paste")
@@
 		)
 		(pad "10" smd roundrect
-			(at -4.65 -5.715 180)
+			(at -4.65 -5.715)
 			(size 2.05 0.6)
 			(layers "B.Cu" "B.Mask" "B.Paste")
@@
 		)
 		(pad "11" smd roundrect
-			(at 4.65 -5.715 180)
+			(at 4.65 -5.715)
 			(size 2.05 0.6)
 			(layers "B.Cu" "B.Mask" "B.Paste")
@@
 		)
 		(pad "12" smd roundrect
-			(at 4.65 -4.445 180)
+			(at 4.65 -4.445)
 			(size 2.05 0.6)
 			(layers "B.Cu" "B.Mask" "B.Paste")
@@
 		)
 		(pad "13" smd roundrect
-			(at 4.65 -3.175 180)
+			(at 4.65 -3.175)
 			(size 2.05 0.6)
 			(layers "B.Cu" "B.Mask" "B.Paste")
@@
 		)
 		(pad "14" smd roundrect
-			(at 4.65 -1.905 180)
+			(at 4.65 -1.905)
 			(size 2.05 0.6)
 			(layers "B.Cu" "B.Mask" "B.Paste")
@@
 		)
 		(pad "15" smd roundrect
-			(at 4.65 -0.635 180)
+			(at 4.65 -0.635)
 			(size 2.05 0.6)
 			(layers "B.Cu" "B.Mask" "B.Paste")
@@
 		)
 		(pad "16" smd roundrect
-			(at 4.65 0.635 180)
+			(at 4.65 0.635)
 			(size 2.05 0.6)
 			(layers "B.Cu" "B.Mask" "B.Paste")
@@
 		)
 		(pad "17" smd roundrect
-			(at 4.65 1.905 180)
+			(at 4.65 1.905)
 			(size 2.05 0.6)
 			(layers "B.Cu" "B.Mask" "B.Paste")
@@
 		)
 		(pad "18" smd roundrect
-			(at 4.65 3.175 180)
+			(at 4.65 3.175)
 			(size 2.05 0.6)
 			(layers "B.Cu" "B.Mask" "B.Paste")
@@
 		)
 		(pad "19" smd roundrect
-			(at 4.65 4.445 180)
+			(at 4.65 4.445)
 			(size 2.05 0.6)
 			(layers "B.Cu" "B.Mask" "B.Paste")
@@
 		)
 		(pad "20" smd roundrect
-			(at 4.65 5.715 180)
+			(at 4.65 5.715)
 			(size 2.05 0.6)
 			(layers "B.Cu" "B.Mask" "B.Paste")

Commit message: Fit the isolated-supply ferrites -- which fixes a supply that was never wired
Asked to integrate the Murata bead the repo owner supplied. Reading the two
isolator pin tables first turned this from an EMC improvement into a defect
fix: the isolated side of BOTH transceivers was unwired.

    CAN_VISOOUT        U3.19 only          dangling
    CAN_VISOIN_OPEN    U3.16 only          dangling
    CAN_ISO_GND        U3.11,12,15,18,20   all merged
    RS485_VISOOUT      U4.12 only          dangling
    RS485_VISOIN_OPEN  U4.19 only          dangling
    RS485_ISO_GND      U4.11,14,16,20      all merged

[10] p.15: "Connect this pin through a ferrite bead and short the PCB trace to
VISOIN FOR OPERATION." [9] p.8: "This pin must be connected externally to
VISOIN." That connection did not exist, so neither bus side had a supply.

Both parts also require the isolated grounds SPLIT, not merged. [10] pins
18,20 GNDISO: "Connect these pins together through one ferrite bead to PCB
ground (bus side)." [9] pins 11,14: "It is recommended to connect Pin 11 and
Pin 14 together through one ferrite bead to PCB ground." And [9] pin 16:
"Ground, Bus Side. DO NOT CONNECT THIS PIN TO PIN 14 AND PIN 11." The
pre-existing net merged exactly the pins that sentence forbids merging.

Four BLM15HD182SN1D fitted -- 1800 ohm at 100 MHz / 2700 ohm at 1 GHz, which
meets [9] p.17's "approximately 2 kohm between the 100 MHz and 1 GHz frequency
range", and is the part [10] Table 12 names by number for this role. Current
rating checked rather than assumed: 200 mA / 2.2 ohm max DCR against
isolated-side transceiver current only, and [9] Table 14 confirms the ADM2582E
has "no current available externally on VISOOUT".

  ERC  0 errors; CAN_VISOOUT and RS485_VISOOUT no longer dangle
  DRC  0 electrical violations

CORRECTION TO THE PREVIOUS COMMIT: it said the ADM3055E "states the reverse
for itself" on ferrites, so the gap was "specifically U4". Wrong. [10] p.25
asks for them just as plainly -- "filter both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
Parts:
- added FB1: BLM15HD182SN1D, L_0402_1005Metric, B.Cu at (40.7, 45.2)
- added FB2: BLM15HD182SN1D, L_0402_1005Metric, B.Cu at (43.2, 45.2)
- added FB3: BLM15HD182SN1D, L_0402_1005Metric, B.Cu at (40.7, 47.2)
- added FB4: BLM15HD182SN1D, L_0402_1005Metric, B.Cu at (43.2, 47.2)
- moved C1 24.0 mm to (28.0, 43.0), turned to -90 degrees
- moved R1 3.50 mm to (24.5, 66.5)
- moved Q1 3.00 mm to (24.0, 52.0)
- moved Q2 3.00 mm to (24.0, 60.0)
- moved R2 2.06 mm to (33.0, 62.5)
- moved Q3 2.00 mm to (32.7, 49.0)
- moved Q4 2.00 mm to (32.5, 56.5)
Connections:
- U3 pad 16: CAN_VISOIN_OPEN -> CAN_VISOIN
- U3 pad 18: CAN_ISO_GND -> CAN_GNDISO
- U3 pad 20: CAN_ISO_GND -> CAN_GNDISO
- U4 pad 11: RS485_ISO_GND -> RS485_GNDISO
- U4 pad 14: RS485_ISO_GND -> RS485_GNDISO
- U4 pad 19: RS485_VISOIN_OPEN -> RS485_VISOIN

Commit message: Add the eight isolated-supply capacitors; stage all twelve parts off-board
The repo owner asked for the remaining isolated-side components to be put
beside the board for hand placement. Done, and the four ferrites from the
previous commit moved out to join them -- the whole group stages together.

    FB1-FB4   staging column at x = 32 mm
    C11-C18   staging column at x = 40 mm
    board outline ends at x = 25.45 mm

Capacitor values and pin pairings are quoted from the datasheets, not chosen:

  [10] p.15 pin 19 VISOOUT : "requires 0.22uF and 10uF capacitors to GNDISO"
  [10] p.15 pin 16 VISOIN  : "requires 0.01uF and 0.1uF decoupling capacitors"
  [9]  p.17                : "0.1 uF and 10 uF for VISOOUT at Pin 11 and Pin
                              12 ... 0.01 uF and 0.1 uF ... for VISOIN at Pin
                              19 and Pin 20"

The two isolated grounds are deliberately not interchangeable: VISOOUT
reservoirs return to the dc-to-dc converter ground (CAN_GNDISO /
RS485_GNDISO), VISOIN decouplers to the bus-side ground (CAN_ISO_GND /
RS485_ISO_GND), and the beads bridge them. Final net topology:

  CAN_VISOOUT    C11.1 C12.1 FB1.1 U3.19
  CAN_GNDISO     C11.2 C12.2 FB2.1 U3.18 U3.20
  CAN_VISOIN     C13.1 C14.1 FB1.2 U3.16
  CAN_ISO_GND    C13.2 C14.2 FB2.2 U3.11 U3.12 U3.15
  RS485_VISOOUT  C15.1 C16.1 FB3.1 U4.12
  RS485_GNDISO   C15.2 C16.2 FB4.1 U4.11 U4.14
  RS485_VISOIN   C17.1 C18.1 FB3.2 U4.19
  RS485_ISO_GND  C17.2 C18.2 FB4.2 U4.16 U4.20

ERC 0 errors. DRC 0 electrical violations. Remaining DRC is 45 silkscreen,
12 drill (12.5.x), 10 starved_thermal on GND.

Package (0805) and voltage rating are AGENTS.md Sec.4 engineering defaults
matching C2..C10. No MPN is claimed for the capacitors -- none has been
selected, and inventing one would be a fabricated citation.

A geometry mistake made and fixed here: the capacitors were first given
horizontal labels at (x +/- 7.62, y), copying the two-terminal R and ferrite
symbols. The generic C symbol is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
Parts:
- added C11: 10uF, C_0805_2012Metric, B.Cu at (59.9, 25.9)
- added C12: 220nF, C_0805_2012Metric, B.Cu at (59.9, 31.4)
- added C13: 100nF, C_0805_2012Metric, B.Cu at (59.9, 36.9)
- added C14: 10nF, C_0805_2012Metric, B.Cu at (59.9, 42.4)
- added C15: 10uF, C_0805_2012Metric, B.Cu at (59.9, 47.9)
- added C16: 100nF, C_0805_2012Metric, B.Cu at (59.9, 53.4)
- added C17: 100nF, C_0805_2012Metric, B.Cu at (59.9, 58.9)
- added C18: 10nF, C_0805_2012Metric, B.Cu at (59.9, 64.4)
- moved FB1 22.3 mm to (51.9, 25.9)
- moved FB2 17.6 mm to (51.9, 29.9)
- moved FB3 17.4 mm to (51.9, 33.9)
- moved FB4 12.7 mm to (51.9, 37.9)
