File: builds/6s/50A/CAN_485_faraday_sameend/kicad/open_secure_esc_6s_50a_can485_faraday_sameend.kicad_pcb (KiCad board)
At the start: 4 copper layers, 32 x 76.1 mm, 65 parts, among them J1 SolderPad_1x04_SMD_P1.27mm_Pr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, J2 SolderPad_1x02_SMD_P2.54mm, J3 SolderPad_1x02_SMD_P2.54mm, J4A SolderWirePad_1x01_SMD_5x10mm, J4B SolderWirePad_1x01_SMD_5x10mm, J4C SolderWirePad_1x01_SMD_5x10mm, J5A SolderWire-6sqmm_1x01_D3.5mm_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, J5B SolderWire-6sqmm_1x01_D3.5mm_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, Q1 Toshiba_2-5W1A_SOP-Advance-N_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, Q2 Toshiba_2-5W1A_SOP-Advance-N_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, Q3 Toshiba_2-5W1A_SOP-Advance-N_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, Q4 Toshiba_2-5W1A_SOP-Advance-N_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, Q5 Toshiba_2-5W1A_SOP-Advance-N_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, Q6 Toshiba_2-5W1A_SOP-Advance-N_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, U1 LQFP-64_10x10mm_P0.5mm, U2 Infineon_PG-USON-10-2-4_3x3mm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, U3 SOIC-20W_7.5x12.8mm_P1.27mm, U4 SOIC-20W_7.5x12.8mm_P1.27mm, U5 TI_RTA0040B_WQFN-40_6x6mm_P0.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, U6 SOIC-8_3.9x4.9mm_P1.27mm, U7 SOIC-8_3.9x4.9mm_P1.27mm, U8 SOIC-8_3.9x4.9mm_P1.27mm

Commit message: cleaned up same-end
Parts:
- moved R7 11.5 mm to (27.0, 85.0)
- moved R12 11.0 mm to (45.0, 85.0)
- moved R5 9.22 mm to (27.0, 72.0)
- moved R13 7.05 mm to (27.0, 74.3)
- moved R10 5.97 mm to (45.0, 72.0)
- moved R4 4.92 mm to (45.0, 74.3), turned to 0 degrees
- moved C3 4.76 mm to (27.0, 82.8)
- moved R8 4.73 mm to (45.0, 82.7)
- moved U2 1.90 mm to (45.4, 79.7)
- moved J1 1.34 mm to (26.0, 79.7)
- moved C9 1.00 mm to (29.9, 65.5)
- moved C10 0.57 mm to (45.0, 76.6)
- moved C4 0.57 mm to (27.0, 76.6)
Changed lines of the file:
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@@
 	(footprint "C_0805_2012Metric"
 		(layer "B.Cu")
-		(at 44.95 76)
+		(at 45.02 76.566)
 		(descr "Capacitor SMD 0805 (2012 Metric), square (rectangular) end terminal, IPC-7351 nominal, (Body size source: IPC-SM-782 page 76, https://www.pcb-3d.com/wordpress/wp-content/uploads/ipc-sm-782a_amendment_1_and_2.pdf, https://docs.google.com/spreadsheets/d/1BsfQQcO9C6DZCsRaXUlFlo91Tg2WpOkGARC1WS5S8t0/edit?usp=sharing), generated with kicad-footprint-generator")
 		(tags "capacitor")
@@
 	(footprint "R_0805_2012Metric"
 		(layer "B.Cu")
-		(at 35.95 69.8 180)
+		(at 27 72 180)
 		(descr "Resistor SMD 0805 (2012 Metric), square (rectangular) end terminal, IPC-7351 nominal, (Body size source: IPC-SM-782 page 72, https://www.pcb-3d.com/wordpress/wp-content/uploads/ipc-sm-782a_amendment_1_and_2.pdf), generated with kicad-footprint-generator")
 		(tags "resistor")
@@
 	(footprint "R_0805_2012Metric"
 		(layer "B.Cu")
-		(at 32.45 69.8 180)
+		(at 27 74.268 180)
 		(descr "Resistor SMD 0805 (2012 Metric), square (rectangular) end terminal, IPC-7351 nominal, (Body size source: IPC-SM-782 page 72, https://www.pcb-3d.com/wordpress/wp-content/uploads/ipc-sm-782a_amendment_1_and_2.pdf), generated with kicad-footprint-generator")
 		(tags "resistor")
@@
 	(footprint "R_0805_2012Metric"
 		(layer "B.Cu")
-		(at 39.45 69.8 180)
+		(at 45 72 180)
 		(descr "Resistor SMD 0805 (2012 Metric), square (rectangular) end terminal, IPC-7351 nominal, (Body size source: IPC-SM-782 page 72, https://www.pcb-3d.com/wordpress/wp-content/uploads/ipc-sm-782a_amendment_1_and_2.pdf), generated with kicad-footprint-generator")
 		(tags "resistor")
@@
 	(footprint "C_0805_2012Metric"
 		(layer "B.Cu")
-		(at 28.95 65.5 180)
+		(at 29.95 65.5 180)
 		(descr "Capacitor SMD 0805 (2012 Metric), square (rectangular) end terminal, IPC-7351 nominal, (Body size source: IPC-SM-782 page 76, https://www.pcb-3d.com/wordpress/wp-content/uploads/ipc-sm-782a_amendment_1_and_2.pdf, https://docs.google.com/spreadsheets/d/1BsfQQcO9C6DZCsRaXUlFlo91Tg2WpOkGARC1WS5S8t0/edit?usp=sharing), generated with kicad-footprint-generator")
 		(tags "capacitor")
@@
 	(footprint "R_0805_2012Metric"
 		(layer "B.Cu")
-		(at 26.95 73.5 180)
+		(at 27 85 180)
 		(descr "Resistor SMD 0805 (2012 Metric), square (rectangular) end terminal, IPC-7351 nominal, (Body size source: IPC-SM-782 page 72, https://www.pcb-3d.com/wordpress/wp-content/uploads/ipc-sm-782a_amendment_1_and_2.pdf), generated with kicad-footprint-generator")
 		(tags "resistor")
@@
 	(footprint "SolderPad_1x04_SMD_P1.27mm_Probe"
 		(layer "B.Cu")
-		(at 25.95 81)
+		(at 26.04 79.664)
 		(descr "SMD PROBE-TARGET pad strip, 4 pads, 1.27 mm pitch, 0.9 x 1.8 mm pads -- a debug-probe landing pattern, NOT a wire-solder pad. For J1 (SWD) only: a bring-up/debug interface, not a flight connection, so it trades solder area for board area. 1.27 mm is the pitch standard pogo-pin debug jigs use, and the strip stays single-row so an off-the-shelf inline fixture fits. Pad geometry is an ENGINEERING DEFAULT (AGENTS.md Sec.4), not a datasheet or IPC value. Do NOT use for J2/J3, which leave the board in service -- see symbols/tools/gen_smd_solder_pad_footprints.py.")
 		(tags "solder pad SMD wire connector 1x04 1.27mm")
@@
 	(footprint "C_0805_2012Metric"
 		(layer "B.Cu")
-		(at 26.95 78 180)
+		(at 26.98 82.762 180)
 		(descr "Capacitor SMD 0805 (2012 Metric), square (rectangular) end terminal, IPC-7351 nominal, (Body size source: IPC-SM-782 page 76, https://www.pcb-3d.com/wordpress/wp-content/uploads/ipc-sm-782a_amendment_1_and_2.pdf, https://docs.google.com/spreadsheets/d/1BsfQQcO9C6DZCsRaXUlFlo91Tg2WpOkGARC1WS5S8t0/edit?usp=sharing), generated with kicad-footprint-generator")
 		(tags "capacitor")
@@
 	(footprint "R_0805_2012Metric"
 		(layer "B.Cu")
-		(at 44.95 74)
+		(at 45 85)
 		(descr "Resistor SMD 0805 (2012 Metric), square (rectangular) end terminal, IPC-7351 nominal, (Body size source: IPC-SM-782 page 72, https://www.pcb-3d.com/wordpress/wp-content/uploads/ipc-sm-782a_amendment_1_and_2.pdf), generated with kicad-footprint-generator")
 		(tags "resistor")
@@
 	(footprint "R_0805_2012Metric"
 		(layer "B.Cu")
-		(at 42.95 69.8 180)
+		(at 45 74.268)
 		(descr "Resistor SMD 0805 (2012 Metric), square (rectangular) end terminal, IPC-7351 nominal, (Body size source: IPC-SM-782 page 72, https://www.pcb-3d.com/wordpress/wp-content/uploads/ipc-sm-782a_amendment_1_and_2.pdf), generated with kicad-footprint-generator")
 		(tags "resistor")
@@
 		(attr smd)
 		(fp_line
-			(start -0.227064 0.735)
-			(end 0.227064 0.735)
+			(start -0.227064 -0.735)
+			(end 0.227064 -0.735)
 			(stroke
 				(width 0.12)
@@
 		)
 		(fp_line
-			(start -0.227064 -0.735)
-			(end 0.227064 -0.735)
+			(start -0.227064 0.735)
+			(end 0.227064 0.735)
 			(stroke
 				(width 0.12)
@@
 		)
 		(fp_line
-			(start 1.68 0.95)
-			(end 1.68 -0.95)
+			(start -1.68 -0.95)
+			(end -1.68 0.95)
 			(stroke
 				(width 0.05)
@@
 		)
 		(fp_line
-			(start 1.68 -0.95)
-			(end -1.68 -0.95)
+			(start -1.68 0.95)
+			(end 1.68 0.95)
 			(stroke
 				(width 0.05)
@@
 		)
 		(fp_line
-			(start -1.68 0.95)
-			(end 1.68 0.95)
+			(start 1.68 -0.95)
+			(end -1.68 -0.95)
 			(stroke
 				(width 0.05)
@@
 		)
 		(fp_line
-			(start -1.68 -0.95)
-			(end -1.68 0.95)
+			(start 1.68 0.95)
+			(end 1.68 -0.95)
 			(stroke
 				(width 0.05)
@@
 		)
 		(fp_line
-			(start 1 0.625)
-			(end 1 -0.625)
+			(start -1 -0.625)
+			(end -1 0.625)
 			(stroke
 				(width 0.1)
@@
 		)
 		(fp_line
-			(start 1 -0.625)
-			(end -1 -0.625)
+			(start -1 0.625)
+			(end 1 0.625)
 			(stroke
 				(width 0.1)
@@
 		)
 		(fp_line
-			(start -1 0.625)
-			(end 1 0.625)
+			(start 1 -0.625)
+			(end -1 -0.625)
 			(stroke
 				(width 0.1)
@@
 		)
 		(fp_line
-			(start -1 -0.625)
-			(end -1 0.625)
+			(start 1 0.625)
+			(end 1 -0.625)
 			(stroke
 				(width 0.1)
@@
 		)
 		(pad "1" smd roundrect
-			(at -0.9125 0 180)
+			(at -0.9125 0)
 			(size 1.025 1.4)
 			(layers "B.Cu" "B.Mask" "B.Paste")
@@
 		)
 		(pad "2" smd roundrect
-			(at 0.9125 0 180)
+			(at 0.9125 0)
 			(size 1.025 1.4)
 			(layers "B.Cu" "B.Mask" "B.Paste")
@@
 	(footprint "R_0805_2012Metric"
 		(layer "B.Cu")
-		(at 44.95 78 180)
+		(at 45 82.732 180)
 		(descr "Resistor SMD 0805 (2012 Metric), square (rectangular) end terminal, IPC-7351 nominal, (Body size source: IPC-SM-782 page 72, https://www.pcb-3d.com/wordpress/wp-content/uploads/ipc-sm-782a_amendment_1_and_2.pdf), generated with kicad-footprint-generator")
 		(tags "resistor")
@@
 	(footprint "C_0805_2012Metric"
 		(layer "B.Cu")
-		(at 26.95 76 180)
+		(at 26.98 76.566 180)
 		(descr "Capacitor SMD 0805 (2012 Metric), square (rectangular) end terminal, IPC-7351 nominal, (Body size source: IPC-SM-782 page 76, https://www.pcb-3d.com/wordpress/wp-content/uploads/ipc-sm-782a_amendment_1_and_2.pdf, https://docs.google.com/spreadsheets/d/1BsfQQcO9C6DZCsRaXUlFlo91Tg2WpOkGARC1WS5S8t0/edit?usp=sharing), generated with kicad-footprint-generator")
 		(tags "capacitor")
@@
 	(footprint "Infineon_PG-USON-10-2-4_3x3mm_P0.5mm_EP1.7x2.5mm"
 		(layer "B.Cu")
-		(at 44.95 81.5 180)
+		(at 45.445 79.664 180)
 		(descr "Infineon PG-USON-10-2,-4, 10-pin USON with exposed thermal pad, 0.5 mm pitch, body 3x3 mm, 0.6 mm max height, EP 1.7x2.5 mm. Package dimensions per REFERENCES.md [45] p.15 Fig.6 / p.16 Fig.7 (Infineon OPTIGA Trust M datasheet, Rev 3.70); land pattern is an IPC-7351-style derivation, NOT an Infineon recommendation (Infineon publishes none) -- see AGENTS.md SS4. Exposed pad is emitted unnumbered: it is n.c. internally and is not a schematic pin. Generated by symbols/tools/gen_optiga_uson10_footprint.py -- do not hand-edit.")
 		(tags "USON DFN PG-USON-10 OPTIGA TrustM Infineon SMD thermal-pad")
