File: builds/6s/50A/CAN_485_faraday_sameend/kicad/open_secure_esc_6s_50a_can485_faraday_sameend.kicad_sch (KiCad schematic)
At the start: 66 parts, among them J1 J_SWD, J2 J_CAN, J3 J_RS485, J4A PH_A_TERM, J4B PH_B_TERM, J4C PH_C_TERM, J5A VM_TERM, J5B GND_TERM, Q1 TPHR8504PL, Q2 TPHR8504PL, Q3 TPHR8504PL, Q4 TPHR8504PL, Q5 TPHR8504PL, Q6 TPHR8504PL, U1 MSPM0G3518_Q1_PM, U2 OPTIGA_TRUST_M, U3 ADM3055E/ADM3057E, U4 ADM2582E/ADM2587E, U5 DRV8353S, U6 INA240, U7 INA240, U8 INA240

Commit message: cleaned up same-end
Parts:
- renumbered J4A to J4A1, J4B to J4B1, J4C to J4C1, J5A to J5A1, J5B to J5B1
Connections:
- net ISENSE_A_HI: no longer Q2.1 (S), Q2.3 (S)
- net ISENSE_B_HI: no longer Q4.1 (S), Q4.3 (S)
- net ISENSE_C_HI: no longer Q6.1 (S), Q6.3 (S)
- net PH_A: no longer Q1.1 (S), Q1.3 (S), Q2.5 (D), Q2.6 (D), Q2.7 (D)
- net PH_B: no longer Q3.1 (S), Q3.3 (S), Q4.5 (D), Q4.6 (D), Q4.7 (D)
- net PH_C: no longer Q5.1 (S), Q5.3 (S), Q6.5 (D), Q6.6 (D), Q6.7 (D)
- net VM: no longer Q1.5 (D), Q1.6 (D), Q1.7 (D), Q3.5 (D), Q3.6 (D), Q3.7 (D), Q5.5 (D), Q5.6 (D), Q5.7 (D)
- new net: Q1.1 (S), Q1.3 (S)
- new net: Q4.1 (S), Q4.3 (S)
- new net: Q2.1 (S), Q2.3 (S)
- new net: Q5.1 (S), Q5.3 (S)
- new net: Q3.1 (S), Q3.3 (S)
- new net: Q6.1 (S), Q6.3 (S)
