File: builds/6s/50A/CAN_485_faraday_sameend/kicad/open_secure_esc_6s_50a_can485_faraday_sameend.kicad_sch (KiCad schematic)
At the start: 66 parts, among them J1 J_SWD, J2 J_CAN, J3 J_RS485, J4A1 PH_A_TERM, J4B1 PH_B_TERM, J4C1 PH_C_TERM, J5A1 VM_TERM, J5B1 GND_TERM, Q1 TPHR8504PL, Q2 TPHR8504PL, Q3 TPHR8504PL, Q4 TPHR8504PL, Q5 TPHR8504PL, Q6 TPHR8504PL, U1 MSPM0G3518_Q1_PM, U2 OPTIGA_TRUST_M, U3 ADM3055E/ADM3057E, U4 ADM2582E/ADM2587E, U5 DRV8353S, U6 INA240, U7 INA240, U8 INA240

Commit message: Stage RHB MCU footprint on-canvas; make RHB the standard MCU package
Two pieces of follow-up to the RHB (VQFN-32) MCU package swap:

- Add the new U1 footprint (Package_DFN_QFN:Texas_RHB0032E_VQFN-32-1EP_
  5x5mm) to each affected .kicad_pcb, replacing the stale LQFP-64
  footprint in place. Every pad is wired to its correct net (verified
  against each board's own net table), but the whole footprint is
  staged OFF-BOARD at fixed clear-of-outline coordinates rather than
  auto-placed or dropped into the old LQFP-64's spot, so final position
  is a manual decision. kicad-cli pcb drc re-run on each board: no new
  violation categories, unconnected-item counts unchanged.

  Done for CAN_485_faraday, CAN_485_faraday_sameend, and
  CAN_485_faraday_sameend_faceted. CAN_485_faraday_faceted's .kicad_pcb
  was left untouched -- it's open in a live, running KiCad GUI session
  (lock file + process observed), and writing to it now risks the next
  GUI save silently discarding the change. Tracked in TODO.md 12.5.bg.

- Swap U1 from MSPM0G3518_Q1_PM to MSPM0G3518_Q1_RHB in the
  CAN_485_faraday_sameend schematic too (same technique as the prior
  commit: identical pin coordinates/types/names, only pin numbers
  change, so existing wiring survives). kicad-cli sch erc re-verified
  at 0 errors, same warning set as before the swap.

- Declare RHB the standard MCU package for all builds going forward in
  README.md and both builds' sym-lib-table descriptions, rather than
  treating the first swap as a one-off.

- New open item (TODO.md 12.5.bg.1): the RHB exposed thermal pad (pad
  33) is left without a net in all three staged footprints -- no
  primary-source confirmation was found that it's internally bonded to
  VSS, so it's marked UNVERIFIED per AGENTS.md Sec.1.3 rather than
  assumed.

Co-Authored-By: Claude Sonnet 5 <noreply@anthropic.com>
Parts:
- U1: value MSPM0G3518_Q1_PM -> MSPM0G3518_Q1_RHB; footprint Package_QFP:LQFP-64_10x10mm_P0.5mm -> Package_DFN_QFN:Texas_RHB0032E_VQFN-32-1EP_5x5mm_P0.5mm_EP3.45x3.45mm; symbol MSPM0G3518_Q1_PM:MSPM0G3518_Q1_PM -> MSPM0G3518_Q1_RHB:MSPM0G3518_Q1_RHB
Connections:
- net 3V3: now also U1.4 (VDD); no longer U1.40 (VDD)
- net ADC_IU: now also U1.28 (ADC_IU); no longer U1.25 (ADC_IU)
- net ADC_IV: now also U1.27 (ADC_IV); no longer U1.24 (ADC_IV)
- net ADC_IW: now also U1.29 (ADC_IW); no longer U1.26 (ADC_IW)
- net GD_SPI_MISO: now also U1.20 (GD_SPI_MISO); no longer U1.2 (GD_SPI_MISO)
- net GND: now also U1.5 (VSS); no longer U1.41 (VSS)
- net NRST: now also U1.3 (NRST); no longer U1.38 (NRST)
- net RS485_DE_RE: now also U1.10 (RS485_DE_RE); no longer U1.37 (RS485_DE_RE)
- net SE_I2C_SCL: now also U1.19 (SE_I2C_SCL); no longer U1.8 (SE_I2C_SCL)
- net SE_RST: now also U1.18 (SE_RST); no longer U1.7 (SE_RST)
- net VBUS_SENSE: now also U1.25 (ADC_VBUS); no longer U1.17 (ADC_VBUS)
- net at U1.1 (RS485_TXD): now also U4.7 (TxD); no longer U5.30 (nSCS)
- net at U1.12 (PWM_AH): now also U5.32 (INHA); no longer J1.1 (Pin_1)
- net at U1.13 (PWM_AL): now also U5.33 (INLA); no longer J1.2 (Pin_2)
- net at U5.28 (SDI): now also U1.22 (GD_SPI_MOSI); no longer U1.3 (GD_SPI_MOSI)
- net at U3.7 (TXD): now also U1.16 (CAN_TX); no longer U1.30 (CAN_TX)
- net at U3.5 (RXD): now also U1.17 (CAN_RX); no longer U1.31 (CAN_RX)
- net at U4.4 (RxD): now also U1.2 (RS485_RXD); no longer U1.34 (RS485_RXD)
- net at U5.29 (SCLK): now also U1.21 (GD_SPI_SCK); no longer U1.4 (GD_SPI_SCK)
- net at U5.36 (INHC): now also U1.14 (PWM_CH); no longer U1.47 (PWM_CH)
- net at U5.37 (INLC): now also U1.15 (PWM_CL); no longer U1.48 (PWM_CL)
- net at U5.34 (INHB): now also U1.7 (PWM_BH); no longer U1.52 (PWM_BH)
- net at U5.35 (INLB): now also U1.8 (PWM_BL); no longer U1.53 (PWM_BL)
- new net: J1.1 (Pin_1), U1.23 (SWDIO)
- new net: J1.2 (Pin_2), U1.24 (SWCLK)
- new net: U1.6 (GD_SPI_CS), U5.30 (nSCS)
Changed lines of the file:
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@@
 	)
 	(symbol
-		(lib_id "MSPM0G3518_Q1_PM:MSPM0G3518_Q1_PM")
+		(lib_id "MSPM0G3518_Q1_RHB:MSPM0G3518_Q1_RHB")
 		(at 529.85 292.54 0)
 		(unit 1)
@@
 			)
 		)
-		(property "Value" "MSPM0G3518_Q1_PM"
+		(property "Value" "MSPM0G3518_Q1_RHB"
 			(at 529.85 278.57 0)
 			(effects
@@
 			)
 		)
-		(property "Footprint" "Package_QFP:LQFP-64_10x10mm_P0.5mm"
+		(property "Footprint" "Package_DFN_QFN:Texas_RHB0032E_VQFN-32-1EP_5x5mm_P0.5mm_EP3.45x3.45mm"
 			(at 529.85 292.54 0)
 			(effects
@@
 			)
 		)
-		(property "Description" "TI MSPM0G3518-Q1 Arm Cortex-M0+ MCU, PM (LQFP-64, 12x12mm) package, orderable M0G3518QPMRQ1 -- project MCU as of 2026-08-10, replacing the NXP S32K144 (REFERENCES.md [31], superseded). Swapped in for its AES-128/256 accelerator with GCM support plus a hardware keystore, which lifts the AES-128 ceiling the S32K144's SHE-compliant CSEc imposed (finding C-01 in docs/secure-element-architecture.md). The Infineon OPTIGA(TM) Trust M secure element (REFERENCES.md [45], schematic U2) is UNAFFECTED by this swap and remains required: the MSPM0's AES engine is symmetric-only, so the Trust M still provides asymmetric PKI device authentication (ECDSA over a fab-provisioned key + X.509 certificate) and ephemeral session-key agreement (ECDHE + KDF), while the MCU consumes the agreed session key for the per-frame authenticated hot path. See docs/secure-element-architecture.md for the full division of labour."
+		(property "Description" "TI MSPM0G3518-Q1 Arm Cortex-M0+ MCU, RHB (VQFN-32, 5x5mm body) package, orderable M0G3518QRHBRQ1 -- swapped 2026-09-06 from the PM (LQFP-64) package (REFERENCES.md [44], same die/part number) to shrink docs/tools/isolation_envelope.py's 'widest non-isolated part' per docs/solutions/architecture-patterns/bom-creepage-audit-can485-faraday.md finding #1. AES-128/256 + GCM accelerator and hardware keystore unaffected by the package change (finding C-01 in docs/secure-element-architecture.md). The Infineon OPTIGA(TM) Trust M secure element (REFERENCES.md [45], schematic U2) remains required and unaffected: the MSPM0's AES engine is symmetric-only, so the Trust M still provides asymmetric PKI device authentication and ephemeral session-key agreement, while the MCU consumes the agreed session key for the per-frame authenticated hot path. See docs/secure-element-architecture.md for the full division of labour."
 			(at 529.85 292.54 0)
 			(effects

Commit message: WIP: stage RHB on the 4th board; fix the 18 FET drain ERC errors
NOTE ON CAN_485_faraday_faceted: this board was open in a live KiCad
GUI session for manual component repositioning (compacting the
layout) while the rest of this branch's work was done, so it was
skipped until the repo owner closed that session. It's now released
and this commit adds the RHB footprint to it -- same treatment as the
other three boards (Package_DFN_QFN:Texas_RHB0032E_VQFN-32-1EP_5x5mm
replacing the stale LQFP-64, every pad wired to its correct net,
staged off-board clear of the board outline for manual placement).

IMPORTANT: the repo owner's manual compaction on this specific board
is IN PROGRESS, not finished ("it needs more work" -- their words).
The committed .kicad_pcb is a snapshot of that in-progress repositioning
plus the staged RHB addition, not a settled layout. Don't treat its
current component placement as final, and don't run any placement
generator against it -- this repo's own rule is never to regenerate a
board after manual packing, and that applies here same as anywhere
else. `kicad-cli pcb drc` confirms the RHB addition itself introduced
no new violations on top of whatever compaction state was already
there (63 violations / 182 unconnected before and after).

Also fixes the 18 pre-existing pin_not_connected ERC errors on
CAN_485_faraday_sameend (Q1-Q6 TPHR8504PL drain pins 5/6/7) flagged by
CI's KiCad ERC/DRC check -- these are pure schematic-connectivity gaps,
independent of any board's component placement, so fixed here rather
than left for after the layout work. Root cause: the FET symbol's
redundant parallel drain pins (5-8, all electrically the same drain
per symbols/specs/TPHR8504PL.json) were left unwired when the symbol
was expanded from an older 3-pin stub to the verified 8-pin version;
only pin 8 carried the real net. Fixed with 3 short wire segments per
FET bussing pins 5-6-7-8 together, each one verified against a
netlist re-export before being trusted -- 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
Connections:
- net PH_A: now also Q2.5 (D), Q2.6 (D), Q2.7 (D)
- net PH_B: now also Q4.5 (D), Q4.6 (D), Q4.7 (D)
- net PH_C: now also Q6.5 (D), Q6.6 (D), Q6.7 (D)
- net VM: now also Q1.5 (D), Q1.6 (D), Q1.7 (D), Q3.5 (D), Q3.6 (D), Q3.7 (D), Q5.5 (D), Q5.6 (D), Q5.7 (D)
Changed lines of the file:
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@@
 		)
+	)
+	(wire
+		(pts
+			(xy 898.58 129.84) (xy 901.12 129.84)
+		)
+		(stroke
+			(width 0)
+			(type default)
+		)
+		(uuid "d5a1f0010-bus0-4000-8000-q1drain001")
+	)
+	(wire
+		(pts
+			(xy 901.12 129.84) (xy 903.66 129.84)
+		)
+		(stroke
+			(width 0)
+			(type default)
+		)
+		(uuid "d5a1f0020-bus0-4000-8000-q1drain002")
+	)
+	(wire
+		(pts
+			(xy 903.66 129.84) (xy 906.1999999999999 129.84)
+		)
+		(stroke
+			(width 0)
+			(type default)
+		)
+		(uuid "d5a1f0030-bus0-4000-8000-q1drain003")
+	)
+	(wire
+		(pts
+			(xy 898.58 169.84) (xy 901.12 169.84)
+		)
+		(stroke
+			(width 0)
+			(type default)
+		)
+		(uuid "d5a1f0040-bus0-4000-8000-q2drain004")
+	)
+	(wire
+		(pts
+			(xy 901.12 169.84) (xy 903.66 169.84)
+		)
+		(stroke
+			(width 0)
+			(type default)
+		)
+		(uuid "d5a1f0050-bus0-4000-8000-q2drain005")
+	)
+	(wire
+		(pts
+			(xy 903.66 169.84) (xy 906.1999999999999 169.84)
+		)
+		(stroke
+			(width 0)
+			(type default)
+		)
+		(uuid "d5a1f0060-bus0-4000-8000-q2drain006")
+	)
+	(wire
+		(pts
+			(xy 898.58 339.84) (xy 901.12 339.84)
+		)
+		(stroke
+			(width 0)
+			(type default)
+		)
+		(uuid "d5a1f0070-bus0-4000-8000-q3drain007")
+	)
+	(wire
+		(pts
+			(xy 901.12 339.84) (xy 903.66 339.84)
+		)
+		(stroke
+			(width 0)
+			(type default)
+		)
+		(uuid "d5a1f0080-bus0-4000-8000-q3drain008")
+	)
+	(wire
+		(pts
+			(xy 903.66 339.84) (xy 906.1999999999999 339.84)
+		)
+		(stroke
+			(width 0)
+			(type default)
+		)
+		(uuid "d5a1f0090-bus0-4000-8000-q3drain009")
+	)
+	(wire
+		(pts
+			(xy 898.58 379.84) (xy 901.12 379.84)
+		)
+		(stroke
+			(width 0)
+			(type default)
+		)
+		(uuid "d5a1f0100-bus0-4000-8000-q4drain010")
+	)
+	(wire
+		(pts
+			(xy 901.12 379.84) (xy 903.66 379.84)
+		)
+		(stroke
+			(width 0)
+			(type default)
+		)
+		(uuid "d5a1f0110-bus0-4000-8000-q4drain011")
+	)
+	(wire
+		(pts
+			(xy 903.66 379.84) (xy 906.1999999999999 379.84)
+		)
+		(stroke
+			(width 0)
+			(type default)
+		)
+		(uuid "d5a1f0120-bus0-4000-8000-q4drain012")
+	)
+	(wire
+		(pts
+			(xy 898.58 549.84) (xy 901.12 549.84)
+		)
+		(stroke
+			(width 0)
+			(type default)
+		)
+		(uuid "d5a1f0130-bus0-4000-8000-q5drain013")
+	)
+	(wire
+		(pts
+			(xy 901.12 549.84) (xy 903.66 549.84)
+		)
+		(stroke
+			(width 0)
+			(type default)
+		)
+		(uuid "d5a1f0140-bus0-4000-8000-q5drain014")
+	)
+	(wire
+		(pts
+			(xy 903.66 549.84) (xy 906.1999999999999 549.84)
+		)
+		(stroke
+			(width 0)
+			(type default)
+		)
+		(uuid "d5a1f0150-bus0-4000-8000-q5drain015")
+	)
+	(wire
+		(pts
+			(xy 898.58 589.84) (xy 901.12 589.84)
+		)
+		(stroke
+			(width 0)
+			(type default)
+		)
+		(uuid "d5a1f0160-bus0-4000-8000-q6drain016")
+	)
+	(wire
+		(pts
+			(xy 901.12 589.84) (xy 903.66 589.84)
+		)
+		(stroke
+			(width 0)
+			(type default)
+		)
+		(uuid "d5a1f0170-bus0-4000-8000-q6drain017")
+	)
+	(wire
+		(pts
+			(xy 903.66 589.84) (xy 906.1999999999999 589.84)
+		)
+		(stroke
+			(width 0)
+			(type default)
+		)
+		(uuid "d5a1f0180-bus0-4000-8000-q6drain018")
 	)
 	(sheet_instances
